File: hardware/Aux_kicker.brd (EAGLE design)
At the start: 23 parts, among them IC2 MIC4429M, IC3 LM324D, Q1 IRF520

Commit message: Changed LED series resistor value to 50k to reflect new break beam
Parts:
- REM: value 10k -> 50k
Changed lines of the file:
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@@
 <attribute name="VALUE" x="53.8688" y="14.2642" size="1.016" layer="27" font="vector" ratio="15" rot="R180"/>
 </element>
-<element name="REM" library="rcl" package="R0805" value="10k" x="15.9532" y="20.9163" smashed="yes" rot="R180">
+<element name="REM" library="rcl" package="R0805" value="50k" x="15.9532" y="20.9163" smashed="yes" rot="R180">
 <attribute name="NAME" x="15.9238" y="23.7877" size="1.016" layer="25" font="vector" ratio="15"/>
 <attribute name="VALUE" x="15.9238" y="22.2637" size="1.016" layer="27" font="vector" ratio="15"/>

Commit message: Minor resistance value changes to aux kicker board
Changed values of resistances in op amp circuit to reflect ones used on
aux kicker boards with new 250V capacitors (instead of 500V capacitors)
Parts:
- R2: value 8.45k -> 5.1k
- R5: value 7.15k -> 15k
Changed lines of the file:
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@@
 <attribute name="VALUE" x="39.243" y="24.892" size="1.016" layer="27" font="vector" ratio="15"/>
 </element>
-<element name="R2" library="rcl" package="R0805" value="8.45k" x="34.544" y="24.892" smashed="yes">
+<element name="R2" library="rcl" package="R0805" value="5.1k" x="34.544" y="24.892" smashed="yes">
 <attribute name="NAME" x="33.909" y="27.686" size="1.016" layer="25" font="vector" ratio="15"/>
 <attribute name="VALUE" x="33.909" y="26.162" size="1.016" layer="27" font="vector" ratio="15"/>
@@
 <attribute name="VALUE" x="46.863" y="21.59" size="1.016" layer="27" font="vector" ratio="15"/>
 </element>
-<element name="R5" library="rcl" package="R0805" value="7.15k" x="41.148" y="20.828" smashed="yes" rot="R90">
+<element name="R5" library="rcl" package="R0805" value="15k" x="41.148" y="20.828" smashed="yes" rot="R90">
 <attribute name="NAME" x="41.783" y="18.288" size="1.016" layer="25" font="vector" ratio="15" rot="R180"/>
 <attribute name="VALUE" x="42.799" y="16.764" size="1.016" layer="27" font="vector" ratio="15" rot="R180"/>
