File: hardware/gen3/MotorConnector/MotorConnector.sch (EAGLE design)
At the start: 19 parts, among them IC1 ATMEGA644A, U1 A4931METTR-T, U2 A4931METTR-T, U3 A4931METTR-T, U4 A4931METTR-T

Commit message: filled in motorboard
Parts:
- removed IC1: ATMEGA644A, atmel:ATMEGA644A
- removed JP1, JP2, JP3, JP4, JP5, JP6, JP7, JP8: M10SILK_FEMALE_PTH, SparkFun-Connectors:M10SILK_FEMALE_PTH
- removed Q1, Q2, Q3, Q4, Q5, Q6: (no value), rfc:N-MOSFET
- removed U1, U2, U3, U4: A4931METTR-T, Allegro_By_element14_Batch_1:A4931METTR-T
- added FRAME1: FRAME-LETTER, SparkFun-Aesthetics:FRAME-LETTER
- added INPUT: M10SILK_FEMALE_PTH, SparkFun-Connectors:M10SILK_FEMALE_PTH
- added QUAD: (no value), con-lstb:MA04-1
- added RIBBON: 53261-11, con-molex:53261-11
Connections:
- new net 5V: INPUT.2, QUAD.1, RIBBON-1.S
- new net GND: INPUT.1, QUAD.3
- new net H1: INPUT.10, RIBBON-3.S
- new net H2: INPUT.9, RIBBON-4.S
- new net H3: INPUT.8, RIBBON-2.S
- new net O1: INPUT.5, RIBBON-10.S, RIBBON-11.S
- new net O2: INPUT.6, RIBBON-8.S, RIBBON-9.S
- new net O3: INPUT.7, RIBBON-6.S, RIBBON-7.S
- new net QEA: INPUT.4, QUAD.2
- new net QEB: INPUT.3, QUAD.4, RIBBON-5.S
Other:
- note added: "5v h3 h1 h2 gnd o3 o2 o1"
