File: hardware/gen3/KickerBoard/KickerBoard.brd (EAGLE design)
At the start: 140 x 132 mm, 87 parts, among them IC1 TL331, Q4 MOSFET-NCHANNELBSS123LT1G, Q6 MOSFET-PCHANNEL, T1 BTV58, U1 NC7WZ08K8X, U2 ATMEGA165PV-8AU

Commit message: changed thyristor to mosfet for simplicity
Parts:
- removed T1: BTV58, triac:TO220CS
- added Q3: MOSFET-NCHANNELFQP30N06L, SparkFun-DiscreteSemi:TO220V
Connections:
- net GND: now also Q3.3; no longer T1.C
- net N$17: now also Q3.2; no longer T1.A
- net N$41: now also Q3.1; no longer T1.G
Changed lines of the file:
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@@
 <?xml version="1.0" encoding="utf-8"?>
 <!DOCTYPE eagle SYSTEM "eagle.dtd">
-<eagle version="6.4">
+<eagle version="7.2.0">
 <drawing>
 <settings>
@@
 <layer number="56" name="wert" color="7" fill="1" visible="no" active="no"/>
 <layer number="57" name="tCAD" color="7" fill="1" visible="no" active="no"/>
-<layer number="90" name="Modules" color="5" fill="1" visible="yes" active="yes"/>
+<layer number="90" name="Modules" color="5" fill="1" visible="no" active="no"/>
 <layer number="91" name="Nets" color="2" fill="1" visible="no" active="no"/>
 <layer number="92" name="Busses" color="1" fill="1" visible="no" active="no"/>
@@
 <pass name="Default">
 <param name="RoutingGrid" value="50mil"/>
+<param name="AutoGrid" value="1"/>
+<param name="Efforts" value="0"/>
+<param name="TopRouterVariant" value="1"/>
 <param name="tpViaShape" value="round"/>
 <param name="PrefDir.1" value="|"/>
@@
 </element>
 <element name="R16" library="rcl" package="R0805" value="LARGE" x="29.05" y="73.19"/>
-<element name="T1" library="triac" package="TO220CS" value="BTV58" x="79.93" y="62.39"/>
 <element name="S2" library="SparkFun-Electromechanical" package="TACTILE-PTH-EZ" value="SWITCH-MOMENTARY-2PTH_EZ" x="69.77" y="57.31"/>
 <element name="FRAME2" library="SparkFun-Aesthetics" package="CREATIVE_COMMONS" value="FRAME-LETTER" x="-77.47" y="85.09"/>
@@
 <element name="LED7" library="SparkFun-LED" package="LED-1206" value="" x="43.02" y="92.24"/>
 <element name="LED8" library="SparkFun-LED" package="LED-1206" value="" x="37.94" y="92.24"/>
+<element name="Q3" library="SparkFun-DiscreteSemi" package="TO220V" value="MOSFET-NCHANNELFQP30N06L" x="-93" y="-31">
+<attribute name="PROD_ID" value="TRANS-10060" x="-93" y="-31" size="1.778" layer="27" display="off"/>
+</element>
 </elements>
 <signals>
@@
 <contactref element="C6" pad="2"/>
 <contactref element="U$3" pad="P$10"/>
-<contactref element="T1" pad="C"/>
 <contactref element="C9" pad="2"/>
 <contactref element="U$4" pad="P$5"/>
@@
 <contactref element="LED7" pad="C"/>
 <contactref element="LED8" pad="C"/>
+<contactref element="Q3" pad="3"/>
 <wire x1="117.05" y1="92.24" x2="120.86" y2="92.24" width="0" layer="19" extent="1-1"/>
 <wire x1="108.64" y1="87.16" x2="117.05" y2="92.24" width="0" layer="19" extent="1-1"/>
@@
 <wire x1="75" y1="92.24" x2="78.45" y2="92.24" width="0" layer="19" extent="1-1"/>
 <wire x1="69.92" y1="92.24" x2="75" y2="92.24" width="0" layer="19" extent="1-1"/>
-<wire x1="37.84" y1="88.24" x2="69.92" y2="92.24" width="0" layer="19" extent="1-1"/>
-<wire x1="59.76" y1="92.24" x2="37.84" y2="88.24" width="0" layer="19" extent="1-1"/>
+<wire x1="59.76" y1="92.24" x2="69.92" y2="92.24" width="0" layer="19" extent="1-1"/>
 <wire x1="54.68" y1="92.24" x2="59.76" y2="92.24" width="0" layer="19" extent="1-1"/>
 <wire x1="49.6" y1="92.24" x2="54.68" y2="92.24" width="0" layer="19" extent="1-1"/>
 <wire x1="44.52" y1="92.24" x2="49.6" y2="92.24" width="0" layer="19" extent="1-1"/>
 <wire x1="39.44" y1="92.24" x2="44.52" y2="92.24" width="0" layer="19" extent="1-1"/>
+<wire x1="37.84" y1="88.24" x2="39.44" y2="92.24" width="0" layer="19" extent="1-1"/>
 <wire x1="33.71" y1="92.24" x2="39.44" y2="92.24" width="0" layer="19" extent="1-1"/>
 <wire x1="29.9" y1="92.24" x2="33.71" y2="92.24" width="0" layer="19" extent="1-1"/>
@@
 <wire x1="88.693" y1="47.15" x2="96.694" y2="47.15" width="0" layer="19" extent="1-1"/>
 <wire x1="79.74" y1="45.88" x2="88.693" y2="47.15" width="0" layer="19" extent="1-1"/>
-<wire x1="77.39" y1="59.85" x2="79.74" y2="45.88" width="0" layer="19" extent="1-1"/>
 <wire x1="91.8934" y1="31.91" x2="88.693" y2="47.15" width="0" layer="19" extent="1-1"/>
+<wire x1="-90.46" y1="-31" x2="32.225" y2="53.6066" width="0" layer="19" extent="1-1"/>
 </signal>
 <signal name="3.3V">
@@
 <signal name="N$17">
 <contactref element="R16" pad="1"/>
-<contactref element="T1" pad="A"/>
-<wire x1="28.1" y1="73.19" x2="79.93" y2="59.85" width="0" layer="19" extent="1-1"/>
+<contactref element="Q3" pad="2"/>
+<wire x1="28.1" y1="73.19" x2="-93" y2="-31" width="0" layer="19" extent="1-1"/>
 </signal>
 <signal name="N$23">
@@
 <contactref element="Q6" pad="3"/>
 <contactref element="R9" pad="2"/>
-<contactref element="T1" pad="G"/>
-<wire x1="82.47" y1="59.85" x2="110.01" y2="82.08" width="0" layer="19" extent="1-1"/>
-<wire x1="66.5188" y1="59.5706" x2="82.47" y2="59.85" width="0" layer="19" extent="1-1"/>
+<contactref element="Q3" pad="1"/>
+<wire x1="66.5188" y1="59.5706" x2="110.01" y2="82.08" width="0" layer="19" extent="1-1"/>
 <wire x1="34.13" y1="80.64" x2="66.5188" y2="59.5706" width="0" layer="19" extent="1-1"/>
+<wire x1="-95.54" y1="-31" x2="34.13" y2="80.64" width="0" layer="19" extent="1-1"/>
 </signal>
 <signal name="N$11">

Commit message: reading in fault pins
Connections:
- net 3.3V: no longer IC1.5, R29.1, U1.8
- net 5V: now also IC1.5, R29.1, U1.8
Changed lines of the file:
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@@
 <contactref element="LOGIC_HEADER" pad="3"/>
 <contactref element="LOGIC_HEADER" pad="4"/>
-<contactref element="U1" pad="8"/>
-<contactref element="IC1" pad="5"/>
-<contactref element="R29" pad="1"/>
 <contactref element="R7" pad="1"/>
 <contactref element="3.3REG" pad="5"/>
@@
 <wire x1="48.1" y1="65.57" x2="64.93" y2="82.1101" width="0" layer="19" extent="1-1"/>
 <wire x1="45.56" y1="65.57" x2="48.1" y2="65.57" width="0" layer="19" extent="1-1"/>
-<wire x1="38.26" y1="74.496" x2="45.56" y2="65.57" width="0" layer="19" extent="1-1"/>
-<wire x1="31.2" y1="79.54" x2="38.26" y2="74.496" width="0" layer="19" extent="1-1"/>
-<wire x1="25.11" y1="87.16" x2="31.2" y2="79.54" width="0" layer="19" extent="1-1"/>
+<wire x1="31.2" y1="79.54" x2="45.56" y2="65.57" width="0" layer="19" extent="1-1"/>
 <wire x1="114.14" y1="65.57" x2="95.99" y2="92.24" width="0" layer="19" extent="1-1"/>
-<wire x1="102.9424" y1="60.612" x2="114.14" y2="65.57" width="0" layer="19" extent="1-1"/>
-<wire x1="97.5068" y1="47.15" x2="102.9424" y2="60.612" width="0" layer="19" extent="1-1"/>
+<wire x1="97.5068" y1="47.15" x2="114.14" y2="65.57" width="0" layer="19" extent="1-1"/>
 <wire x1="91.106" y1="31.91" x2="97.5068" y2="47.15" width="0" layer="19" extent="1-1"/>
 </signal>
@@
 <contactref element="LOGIC_HEADER" pad="5"/>
 <contactref element="LOGIC_HEADER" pad="6"/>
+<contactref element="R29" pad="1"/>
+<contactref element="U1" pad="8"/>
+<contactref element="IC1" pad="5"/>
 <wire x1="61.12" y1="82.1101" x2="81.25" y2="92.24" width="0" layer="19" extent="1-1"/>
 <wire x1="53.18" y1="65.57" x2="61.12" y2="82.1101" width="0" layer="19" extent="1-1"/>
 <wire x1="50.64" y1="65.57" x2="53.18" y2="65.57" width="0" layer="19" extent="1-1"/>
+<wire x1="38.26" y1="74.496" x2="50.64" y2="65.57" width="0" layer="19" extent="1-1"/>
+<wire x1="25.11" y1="87.16" x2="38.26" y2="74.496" width="0" layer="19" extent="1-1"/>
+<wire x1="102.9424" y1="60.612" x2="81.25" y2="92.24" width="0" layer="19" extent="1-1"/>
 </signal>
 <signal name="N$19">

Commit message: hooked up ss lines
Connections:
- net SS1 renamed SS_M
- net SS3 renamed SS_E1
- net SS4 renamed SS_E2
- net SS5 renamed SS_E3
- removed net SS2: SPI_HEADER.5
- new net SS_K: SPI_HEADER.5, U2.11
- net SCK: no longer U2.11
Changed lines of the file:
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@@
 <contactref element="R4" pad="1"/>
 <contactref element="PROG_CNT" pad="3"/>
-<contactref element="U2" pad="11"/>
 <wire x1="116.68" y1="63.03" x2="105.62" y2="92.24" width="0" layer="19" extent="1-1"/>
-<wire x1="86.28" y1="37.5234" x2="116.68" y2="63.03" width="0" layer="19" extent="1-1"/>
 </signal>
-<signal name="SS1">
+<signal name="SS_M">
 <contactref element="SPI_HEADER" pad="4"/>
 </signal>
-<signal name="SS2">
+<signal name="SS_K">
 <contactref element="SPI_HEADER" pad="5"/>
+<contactref element="U2" pad="11"/>
+<wire x1="86.28" y1="37.5234" x2="55.72" y2="74.46" width="0" layer="19" extent="1-1"/>
 </signal>
-<signal name="SS3">
+<signal name="SS_E1">
 <contactref element="SPI_HEADER" pad="6"/>
 </signal>
-<signal name="SS4">
+<signal name="SS_E2">
 <contactref element="SPI_HEADER" pad="7"/>
 </signal>
-<signal name="SS5">
+<signal name="SS_E3">
 <contactref element="SPI_HEADER" pad="8"/>
 </signal>

Commit message: fixed ERCs on all boards
Parts:
- removed R10: (no value), resistor:R0805
- C82: value (none) -> 100pF
- renumbered C8100PF to C82
Connections:
- removed net DISCHARGE: U2.50
- removed net N$20: BATT.2
- new net DONE: R7.2, U$4.P$2, U2.46
- net 12VGND: now also BATT.2, Q3.3, R9.1, U$3.P$10
- net CHARGE: no longer R10.1
- net GND: no longer Q3.3, R10.2, R9.1, U$3.P$10
- net N$12: now also R2.2, SPI_HEADER.1; no longer R7.2, U$4.P$2
- net N$19: now also S1.2
- net ~DIS: now also U2.50
Changed lines of the file:
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@@
 </element>
 <element name="U$2" library="SparkFun-DiscreteSemi" package="SMA-DIODE" value="TVS" x="114.14" y="87.16"/>
-<element name="R10" library="resistor" package="R0805" value="" x="107.79" y="87.16"/>
 <element name="R11" library="resistor" package="R0805" value="20m" x="69.69" y="80.81"/>
-<element name="C8100PF" library="rcl" package="C0805" value="" x="53.18" y="79.54"/>
+<element name="C82" library="rcl" package="C0805" value="100pF" x="53.18" y="79.54"/>
 <element name="C9" library="rcl" package="C0805" value="10uF" x="114.14" y="82.08"/>
 <element name="C3" library="rcl" package="C0805" value="47uF" x="22.7" y="73.19"/>
@@
 <contactref element="U1" pad="4"/>
 <contactref element="C6" pad="2"/>
-<contactref element="U$3" pad="P$10"/>
 <contactref element="C9" pad="2"/>
 <contactref element="U$4" pad="P$5"/>
-<contactref element="C8100PF" pad="2"/>
+<contactref element="C82" pad="2"/>
 <contactref element="R6" pad="2"/>
 <contactref element="R11" pad="2"/>
 <contactref element="C3" pad="2"/>
 <contactref element="C5" pad="2"/>
-<contactref element="R10" pad="2"/>
-<contactref element="R9" pad="1"/>
 <contactref element="C8" pad="2"/>
 <contactref element="C7" pad="2"/>
@@
 <contactref element="LED7" pad="C"/>
 <contactref element="LED8" pad="C"/>
-<contactref element="Q3" pad="3"/>
 <wire x1="117.05" y1="92.24" x2="120.86" y2="92.24" width="0" layer="19" extent="1-1"/>
-<wire x1="108.64" y1="87.16" x2="117.05" y2="92.24" width="0" layer="19" extent="1-1"/>
-<wire x1="104.11" y1="87.16" x2="108.64" y2="87.16" width="0" layer="19" extent="1-1"/>
-<wire x1="108.11" y1="82.08" x2="108.64" y2="87.16" width="0" layer="19" extent="1-1"/>
-<wire x1="115.09" y1="82.08" x2="108.11" y2="82.08" width="0" layer="19" extent="1-1"/>
-<wire x1="121.44" y1="82.08" x2="115.09" y2="82.08" width="0" layer="19" extent="1-1"/>
+<wire x1="121.44" y1="82.08" x2="120.86" y2="92.24" width="0" layer="19" extent="1-1"/>
+<wire x1="115.09" y1="82.08" x2="121.44" y2="82.08" width="0" layer="19" extent="1-1"/>
+<wire x1="104.11" y1="87.16" x2="115.09" y2="82.08" width="0" layer="19" extent="1-1"/>
 <wire x1="92.18" y1="92.24" x2="104.11" y2="87.16" width="0" layer="19" extent="1-1"/>
 <wire x1="84.8" y1="92.24" x2="92.18" y2="92.24" width="0" layer="19" extent="1-1"/>
@@
 <wire x1="96.694" y1="47.15" x2="100.0976" y2="59.088" width="0" layer="19" extent="1-1"/>
 <wire x1="88.693" y1="47.15" x2="96.694" y2="47.15" width="0" layer="19" extent="1-1"/>
-<wire x1="79.74" y1="45.88" x2="88.693" y2="47.15" width="0" layer="19" extent="1-1"/>
 <wire x1="91.8934" y1="31.91" x2="88.693" y2="47.15" width="0" layer="19" extent="1-1"/>
-<wire x1="-90.46" y1="-31" x2="32.225" y2="53.6066" width="0" layer="19" extent="1-1"/>
 </signal>
 <signal name="3.3V">
@@
 <contactref element="U$4" pad="P$4"/>
 <contactref element="U$4" pad="P$1"/>
-<contactref element="U$3" pad="P$5"/>
 <contactref element="U$3" pad="P$4"/>
 <contactref element="C9" pad="1"/>
@@
 <contactref element="3.3REG" pad="1"/>
 <contactref element="S1" pad="3"/>
+<contactref element="U$3" pad="P$5"/>
 <wire x1="113.19" y1="82.08" x2="119.54" y2="82.08" width="0" layer="19" extent="1-1"/>
 <wire x1="119.22" y1="74.46" x2="119.54" y2="82.08" width="0" layer="19" extent="1-1"/>
@@
 <contactref element="C1" pad="-"/>
 <contactref element="C2" pad="-"/>
+<contactref element="BATT" pad="2"/>
+<contactref element="U$3" pad="P$10"/>
+<contactref element="R9" pad="1"/>
+<contactref element="Q3" pad="3"/>
 <wire x1="90.38" y1="92.24" x2="98" y2="92.24" width="0" layer="19" extent="1-1"/>
 <wire x1="105.25" y1="80.81" x2="98" y2="92.24" width="0" layer="19" extent="1-1"/>
+<wire x1="108.11" y1="82.08" x2="105.25" y2="80.81" width="0" layer="19" extent="1-1"/>
 <wire x1="106.52" y1="74.46" x2="105.25" y2="80.81" width="0" layer="19" extent="1-1"/>
 <wire x1="109.06" y1="74.46" x2="106.52" y2="74.46" width="0" layer="19" extent="1-1"/>
@@
 <wire x1="101.44" y1="74.46" x2="103.98" y2="74.46" width="0" layer="19" extent="1-1"/>
 <wire x1="98.9" y1="74.46" x2="101.44" y2="74.46" width="0" layer="19" extent="1-1"/>
+<wire x1="93.86" y1="58.58" x2="98.9" y2="74.46" width="0" layer="19" extent="1-1"/>
+<wire x1="79.74" y1="45.88" x2="93.86" y2="58.58" width="0" layer="19" extent="1-1"/>
 <wire x1="65.88" y1="79.5099" x2="90.38" y2="92.24" width="0" layer="19" extent="1-1"/>
 <wire x1="62.07" y1="79.5099" x2="65.88" y2="79.5099" width="0" layer="19" extent="1-1"/>
@@
 <wire x1="38.07" y1="87.16" x2="42.7" y2="78.54" width="0" layer="19" extent="1-1"/>
 <wire x1="32.99" y1="87.16" x2="38.07" y2="87.16" width="0" layer="19" extent="1-1"/>
-<wire x1="38.02" y1="29.37" x2="42.7" y2="78.54" width="0" layer="19" extent="1-1"/>
-<wire x1="50.72" y1="29.37" x2="38.02" y2="29.37" width="0" layer="19" extent="1-1"/>
+<wire x1="50.72" y1="29.37" x2="79.74" y2="45.88" width="0" layer="19" extent="1-1"/>
+<wire x1="38.02" y1="29.37" x2="50.72" y2="29.37" width="0" layer="19" extent="1-1"/>
 <wire x1="68.5" y1="9.05" x2="50.72" y2="29.37" width="0" layer="19" extent="1-1"/>
 <wire x1="105.33" y1="9.05" x2="68.5" y2="9.05" width="0" layer="19" extent="1-1"/>
+<wire x1="-90.46" y1="-31" x2="38.02" y2="29.37" width="0" layer="19" extent="1-1"/>
 </signal>
 <signal name="N$5">
 <contactref element="U$3" pad="P$7"/>
-<contactref element="U$3" pad="P$6"/>
 <contactref element="R5" pad="2"/>
 <contactref element="Q5" pad="DRAIN"/>
 <contactref element="R8" pad="2"/>
+<contactref element="U$3" pad="P$6"/>
 <wire x1="89.59" y1="80.81" x2="97.21" y2="80.81" width="0" layer="19" extent="1-1"/>
-<wire x1="20.16" y1="55.41" x2="89.59" y2="80.81" width="0" layer="19" extent="1-1"/>
 <wire x1="79.74" y1="34.63" x2="89.59" y2="80.81" width="0" layer="19" extent="1-1"/>
 <wire x1="79.74" y1="30.88" x2="79.74" y2="34.63" width="0" layer="19" extent="1-1"/>
+<wire x1="20.16" y1="55.41" x2="79.74" y2="34.63" width="0" layer="19" extent="1-1"/>
 </signal>
 <signal name="N$8">
@@
 <wire x1="22.675" y1="87.275" x2="87.89" y2="80.81" width="0" layer="19" extent="1-1"/>
 </signal>
-<signal name="N$12">
+<signal name="DONE">
 <contactref element="R7" pad="2"/>
 <contactref element="U$4" pad="P$2"/>
+<contactref element="U2" pad="46"/>
+<wire x1="101.52" y1="43.9242" x2="83.24" y2="80.81" width="0" layer="19" extent="1-1"/>
 <wire x1="18.405" y1="87.775" x2="83.24" y2="80.81" width="0" layer="19" extent="1-1"/>
 </signal>
@@
 <signal name="CHARGE">
 <contactref element="U$4" pad="P$3"/>
-<contactref element="R10" pad="1"/>
 <contactref element="U2" pad="51"/>
-<wire x1="98.2942" y1="47.15" x2="106.94" y2="87.16" width="0" layer="19" extent="1-1"/>
-<wire x1="18.405" y1="87.275" x2="106.94" y2="87.16" width="0" layer="19" extent="1-1"/>
+<wire x1="18.405" y1="87.275" x2="98.2942" y2="47.15" width="0" layer="19" extent="1-1"/>
 </signal>
 <signal name="N$24">
@@
 <contactref element="R6" pad="1"/>
 <contactref element="U$4" pad="P$10"/>
-<contactref element="C8100PF" pad="1"/>
+<contactref element="C82" pad="1"/>
 <wire x1="52.23" y1="79.54" x2="75.19" y2="80.81" width="0" layer="19" extent="1-1"/>
 <wire x1="22.675" y1="88.275" x2="52.23" y2="79.54" width="0" layer="19" extent="1-1"/>
@@
 <contactref element="D2" pad="C"/>
 <wire x1="30" y1="73.19" x2="105.59" y2="65.57" width="0" layer="19" extent="1-1"/>
-</signal>
-<signal name="DISCHARGE">
-<contactref element="U2" pad="50"/>
 </signal>
 <signal name="DRIB">
@@
 <signal name="N$19">
 <contactref element="BATT" pad="1"/>
-</signal>
-<signal name="N$20">
-<contactref element="BATT" pad="2"/>
+<contactref element="S1" pad="2"/>
+<wire x1="24.05" y1="34.45" x2="88.86" y2="58.58" width="0" layer="19" extent="1-1"/>
 </signal>
 <signal name="GLED1">
@@
 <signal name="~DIS">
 <contactref element="Q6" pad="1"/>
+<contactref element="U2" pad="50"/>
+<wire x1="33.18" y1="78.54" x2="99.107" y2="47.15" width="0" layer="19" extent="1-1"/>
 </signal>
 <signal name="N$41">
@@
 <wire x1="36.44" y1="92.24" x2="55.59" y2="87.16" width="0" layer="19" extent="1-1"/>
 </signal>
+<signal name="N$12">
+<contactref element="R2" pad="2"/>
+<contactref element="SPI_HEADER" pad="1"/>
+<wire x1="45.56" y1="74.46" x2="115.04" y2="92.24" width="0" layer="19" extent="1-1"/>
+</signal>
 </signals>

Commit message: discharge resistor value
Parts:
- R16: value LARGE -> 2k, 5w
Changed lines of the file:
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@@
 <attribute name="STOREFRONT_ID" value="PRT-08432" x="137" y="-50" size="1.778" layer="27" display="off"/>
 </element>
-<element name="R16" library="rcl" package="R0805" value="LARGE" x="29.05" y="73.19"/>
+<element name="R16" library="rcl" package="R0805" value="2k, 5w" x="29.05" y="73.19"/>
 <element name="S2" library="SparkFun-Electromechanical" package="TACTILE-PTH-EZ" value="SWITCH-MOMENTARY-2PTH_EZ" x="69.77" y="57.31"/>
 <element name="FRAME2" library="SparkFun-Aesthetics" package="CREATIVE_COMMONS" value="FRAME-LETTER" x="-77.47" y="85.09"/>

Commit message: decoupling
Parts:
- added C13, C14, C15, C16: .1uF, SparkFun-Capacitors:1206
- C10, C11: value >2.2uF -> 100uF
Connections:
- net 12V: now also C16.1
- net 12VGND: now also C16.2
- net 3.3V: now also C13.1
- net 5V: now also C14.1, C15.1
- net GND: now also C13.2, C14.2, C15.2
Changed lines of the file:
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@@
 <element name="TMP" library="SparkFun-Passives" package="0805" value="0" x="91.28" y="92.24"/>
 <element name="S1" library="switch" package="M9040P" value="" x="24.05" y="34.45"/>
-<element name="C10" library="SparkFun-Capacitors" package="EIA3216" value="&gt;2.2uF" x="86.2" y="92.24">
+<element name="C10" library="SparkFun-Capacitors" package="EIA3216" value="100uF" x="86.2" y="92.24">
 <attribute name="PROD_ID" value="CAP-00811" x="137" y="-50" size="1.778" layer="27" display="off"/>
 </element>
-<element name="C11" library="SparkFun-Capacitors" package="EIA3216" value="&gt;2.2uF" x="79.85" y="92.24">
+<element name="C11" library="SparkFun-Capacitors" package="EIA3216" value="100uF" x="79.85" y="92.24">
 <attribute name="PROD_ID" value="CAP-00811" x="137" y="-50" size="1.778" layer="27" display="off"/>
 </element>
@@
 <attribute name="PROD_ID" value="TRANS-10060" x="-93" y="-31" size="1.778" layer="27" display="off"/>
 </element>
+<element name="C13" library="SparkFun-Capacitors" package="1206" value=".1uF" x="-95" y="-37"/>
+<element name="C14" library="SparkFun-Capacitors" package="1206" value=".1uF" x="-95" y="-41"/>
+<element name="C15" library="SparkFun-Capacitors" package="1206" value=".1uF" x="-95" y="-45"/>
+<element name="C16" library="SparkFun-Capacitors" package="1206" value=".1uF" x="-95" y="-49"/>
 </elements>
 <signals>
@@
 <contactref element="LED7" pad="C"/>
 <contactref element="LED8" pad="C"/>
+<contactref element="C14" pad="2"/>
+<contactref element="C13" pad="2"/>
+<contactref element="C15" pad="2"/>
 <wire x1="117.05" y1="92.24" x2="120.86" y2="92.24" width="0" layer="19" extent="1-1"/>
 <wire x1="121.44" y1="82.08" x2="120.86" y2="92.24" width="0" layer="19" extent="1-1"/>
@@
 <wire x1="88.693" y1="47.15" x2="96.694" y2="47.15" width="0" layer="19" extent="1-1"/>
 <wire x1="91.8934" y1="31.91" x2="88.693" y2="47.15" width="0" layer="19" extent="1-1"/>
+<wire x1="-93.6" y1="-37" x2="32.225" y2="53.6066" width="0" layer="19" extent="1-1"/>
+<wire x1="-93.6" y1="-41" x2="-93.6" y2="-37" width="0" layer="19" extent="1-1"/>
+<wire x1="-93.6" y1="-45" x2="-93.6" y2="-41" width="0" layer="19" extent="1-1"/>
 </signal>
 <signal name="3.3V">
@@
 <contactref element="U2" pad="21"/>
 <contactref element="U2" pad="52"/>
+<contactref element="C13" pad="1"/>
 <wire x1="87.6" y1="92.24" x2="95.99" y2="92.24" width="0" layer="19" extent="1-1"/>
 <wire x1="81.54" y1="80.81" x2="87.6" y2="92.24" width="0" layer="19" extent="1-1"/>
@@
 <wire x1="97.5068" y1="47.15" x2="114.14" y2="65.57" width="0" layer="19" extent="1-1"/>
 <wire x1="91.106" y1="31.91" x2="97.5068" y2="47.15" width="0" layer="19" extent="1-1"/>
+<wire x1="-96.4" y1="-37" x2="31.2" y2="79.54" width="0" layer="19" extent="1-1"/>
 </signal>
 <signal name="MOSI">
@@
 <contactref element="S1" pad="3"/>
 <contactref element="U$3" pad="P$5"/>
+<contactref element="C16" pad="1"/>
 <wire x1="113.19" y1="82.08" x2="119.54" y2="82.08" width="0" layer="19" extent="1-1"/>
 <wire x1="119.22" y1="74.46" x2="119.54" y2="82.08" width="0" layer="19" extent="1-1"/>
@@
 <wire x1="57.07" y1="30.88" x2="24.05" y2="29.751" width="0" layer="19" extent="1-1"/>
 <wire x1="57.07" y1="34.63" x2="57.07" y2="30.88" width="0" layer="19" extent="1-1"/>
+<wire x1="-96.4" y1="-49" x2="24.05" y2="29.751" width="0" layer="19" extent="1-1"/>
 </signal>
 <signal name="12VGND">
@@
 <contactref element="R9" pad="1"/>
 <contactref element="Q3" pad="3"/>
+<contactref element="C16" pad="2"/>
 <wire x1="90.38" y1="92.24" x2="98" y2="92.24" width="0" layer="19" extent="1-1"/>
 <wire x1="105.25" y1="80.81" x2="98" y2="92.24" width="0" layer="19" extent="1-1"/>
@@
 <wire x1="105.33" y1="9.05" x2="68.5" y2="9.05" width="0" layer="19" extent="1-1"/>
 <wire x1="-90.46" y1="-31" x2="38.02" y2="29.37" width="0" layer="19" extent="1-1"/>
+<wire x1="-93.6" y1="-49" x2="-90.46" y2="-31" width="0" layer="19" extent="1-1"/>
 </signal>
 <signal name="N$5">
@@
 <contactref element="U1" pad="8"/>
 <contactref element="IC1" pad="5"/>
+<contactref element="C14" pad="1"/>
+<contactref element="C15" pad="1"/>
 <wire x1="61.12" y1="82.1101" x2="81.25" y2="92.24" width="0" layer="19" extent="1-1"/>
 <wire x1="53.18" y1="65.57" x2="61.12" y2="82.1101" width="0" layer="19" extent="1-1"/>
@@
 <wire x1="25.11" y1="87.16" x2="38.26" y2="74.496" width="0" layer="19" extent="1-1"/>
 <wire x1="102.9424" y1="60.612" x2="81.25" y2="92.24" width="0" layer="19" extent="1-1"/>
+<wire x1="-96.4" y1="-41" x2="25.11" y2="87.16" width="0" layer="19" extent="1-1"/>
+<wire x1="-96.4" y1="-45" x2="-96.4" y2="-41" width="0" layer="19" extent="1-1"/>
 </signal>
 <signal name="N$19">
