File: hardware/gen3/KickerBoard/KickerBoard.brd (EAGLE design)
At the start: 140 x 132 mm, 90 parts, among them IC1 TL331, Q3 MOSFET-NCHANNELFQP30N06L, Q4 MOSFET-NCHANNELBSS123LT1G, Q6 MOSFET-PCHANNEL, U1 NC7WZ08K8X, U2 ATMEGA165PV-8AU

Commit message: fixed current limiting
Parts:
- C12, C4: value 100nF -> .1uF
Changed lines of the file:
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@@
 <attribute name="PROD_ID" value="TRANS-08285" x="137" y="-50" size="1.778" layer="27" display="off"/>
 </element>
-<element name="C4" library="SparkFun-Capacitors" package="0805" value="100nF" x="121.76" y="92.24"/>
-<element name="C12" library="SparkFun-Capacitors" package="0805" value="100nF" x="117.95" y="92.24"/>
+<element name="C4" library="SparkFun-Capacitors" package="0805" value=".1uF" x="121.76" y="92.24"/>
+<element name="C12" library="SparkFun-Capacitors" package="0805" value=".1uF" x="117.95" y="92.24"/>
 <element name="R30" library="SparkFun-Passives" package="0805" value="10k" x="95.09" y="92.24"/>
 <element name="U2" library="Atmel_By_element14_Batch_1-00" package="QFP80P1600X1600X120-64N" value="ATMEGA165PV-8AU" x="93.9" y="39.53">

Commit message: Added programmer port to boards
Parts:
- removed PROG_CNT: (no value), SparkFun-Connectors:2X3
- added JP1: M05X2PTH, SparkFun-Connectors:AVR_ICSP
Connections:
- net 3.3V: now also JP1.2; no longer PROG_CNT.2
- net GND: now also JP1.10, JP1.4, JP1.6, JP1.8; no longer PROG_CNT.6
- net MISO: now also JP1.9; no longer PROG_CNT.1
- net MOSI: now also JP1.1; no longer PROG_CNT.4
- net RESET: now also JP1.5; no longer PROG_CNT.5
- net SCK: now also JP1.7; no longer PROG_CNT.3
Changed lines of the file:
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@@
 <element name="R3" library="SparkFun-Passives" package="0805" value="10k" x="110.33" y="92.24"/>
 <element name="R4" library="SparkFun-Passives" package="0805" value="10k" x="106.52" y="92.24"/>
-<element name="PROG_CNT" library="SparkFun-Connectors" package="2X3" value="" x="114.14" y="63.03">
-<attribute name="PROD_ID" value="CONN-09701" x="137" y="-50" size="1.778" layer="27" display="off"/>
-</element>
 <element name="U$3" library="kickerchips" package="10-TRANSFORMER" value="32052-TRANSFORMER" x="57.07" y="45.88"/>
 <element name="Q5" library="rfc" package="DPAK" value="" x="20.16" y="55.41"/>
@@
 <element name="C15" library="SparkFun-Capacitors" package="1206" value=".1uF" x="-95" y="-45"/>
 <element name="C16" library="SparkFun-Capacitors" package="1206" value=".1uF" x="-95" y="-49"/>
+<element name="JP1" library="SparkFun-Connectors" package="AVR_ICSP" value="M05X2PTH" x="-101" y="-44"/>
 </elements>
 <signals>
 <signal name="GND">
-<contactref element="PROG_CNT" pad="6"/>
 <contactref element="LOGIC_HEADER" pad="1"/>
 <contactref element="LOGIC_HEADER" pad="2"/>
@@
 <contactref element="C13" pad="2"/>
 <contactref element="C15" pad="2"/>
+<contactref element="JP1" pad="10"/>
+<contactref element="JP1" pad="8"/>
+<contactref element="JP1" pad="6"/>
+<contactref element="JP1" pad="4"/>
 <wire x1="117.05" y1="92.24" x2="120.86" y2="92.24" width="0" layer="19" extent="1-1"/>
 <wire x1="121.44" y1="82.08" x2="120.86" y2="92.24" width="0" layer="19" extent="1-1"/>
@@
 <wire x1="34.765" y1="53.6066" x2="40.48" y2="65.57" width="0" layer="19" extent="1-1"/>
 <wire x1="32.225" y1="53.6066" x2="34.765" y2="53.6066" width="0" layer="19" extent="1-1"/>
-<wire x1="119.22" y1="65.57" x2="121.44" y2="82.08" width="0" layer="19" extent="1-1"/>
-<wire x1="100.0976" y1="59.088" x2="119.22" y2="65.57" width="0" layer="19" extent="1-1"/>
+<wire x1="100.0976" y1="59.088" x2="115.09" y2="82.08" width="0" layer="19" extent="1-1"/>
 <wire x1="96.694" y1="47.15" x2="100.0976" y2="59.088" width="0" layer="19" extent="1-1"/>
 <wire x1="88.693" y1="47.15" x2="96.694" y2="47.15" width="0" layer="19" extent="1-1"/>
@@
 <wire x1="-93.6" y1="-41" x2="-93.6" y2="-37" width="0" layer="19" extent="1-1"/>
 <wire x1="-93.6" y1="-45" x2="-93.6" y2="-41" width="0" layer="19" extent="1-1"/>
+<wire x1="-99.73" y1="-41.46" x2="-93.6" y2="-41" width="0" layer="19" extent="1-1"/>
+<wire x1="-99.73" y1="-44" x2="-99.73" y2="-41.46" width="0" layer="19" extent="1-1"/>
+<wire x1="-99.73" y1="-46.54" x2="-99.73" y2="-44" width="0" layer="19" extent="1-1"/>
+<wire x1="-99.73" y1="-49.08" x2="-99.73" y2="-46.54" width="0" layer="19" extent="1-1"/>
 </signal>
 <signal name="3.3V">
-<contactref element="PROG_CNT" pad="2"/>
 <contactref element="LOGIC_HEADER" pad="3"/>
 <contactref element="LOGIC_HEADER" pad="4"/>
@@
 <contactref element="U2" pad="52"/>
 <contactref element="C13" pad="1"/>
+<contactref element="JP1" pad="2"/>
 <wire x1="87.6" y1="92.24" x2="95.99" y2="92.24" width="0" layer="19" extent="1-1"/>
 <wire x1="81.54" y1="80.81" x2="87.6" y2="92.24" width="0" layer="19" extent="1-1"/>
@@
 <wire x1="45.56" y1="65.57" x2="48.1" y2="65.57" width="0" layer="19" extent="1-1"/>
 <wire x1="31.2" y1="79.54" x2="45.56" y2="65.57" width="0" layer="19" extent="1-1"/>
-<wire x1="114.14" y1="65.57" x2="95.99" y2="92.24" width="0" layer="19" extent="1-1"/>
-<wire x1="97.5068" y1="47.15" x2="114.14" y2="65.57" width="0" layer="19" extent="1-1"/>
+<wire x1="97.5068" y1="47.15" x2="81.54" y2="80.81" width="0" layer="19" extent="1-1"/>
 <wire x1="91.106" y1="31.91" x2="97.5068" y2="47.15" width="0" layer="19" extent="1-1"/>
 <wire x1="-96.4" y1="-37" x2="31.2" y2="79.54" width="0" layer="19" extent="1-1"/>
+<wire x1="-99.73" y1="-38.92" x2="-96.4" y2="-37" width="0" layer="19" extent="1-1"/>
 </signal>
 <signal name="MOSI">
 <contactref element="R2" pad="1"/>
-<contactref element="PROG_CNT" pad="4"/>
 <contactref element="U2" pad="12"/>
-<wire x1="116.68" y1="65.57" x2="113.24" y2="92.24" width="0" layer="19" extent="1-1"/>
-<wire x1="86.28" y1="36.736" x2="116.68" y2="65.57" width="0" layer="19" extent="1-1"/>
+<contactref element="JP1" pad="1"/>
+<wire x1="86.28" y1="36.736" x2="113.24" y2="92.24" width="0" layer="19" extent="1-1"/>
+<wire x1="-102.27" y1="-38.92" x2="86.28" y2="36.736" width="0" layer="19" extent="1-1"/>
 </signal>
 <signal name="MISO">
 <contactref element="R3" pad="1"/>
-<contactref element="PROG_CNT" pad="1"/>
 <contactref element="U2" pad="13"/>
-<wire x1="114.14" y1="63.03" x2="109.43" y2="92.24" width="0" layer="19" extent="1-1"/>
-<wire x1="86.28" y1="35.9232" x2="114.14" y2="63.03" width="0" layer="19" extent="1-1"/>
+<contactref element="JP1" pad="9"/>
+<wire x1="86.28" y1="35.9232" x2="109.43" y2="92.24" width="0" layer="19" extent="1-1"/>
+<wire x1="-102.27" y1="-49.08" x2="86.28" y2="35.9232" width="0" layer="19" extent="1-1"/>
 </signal>
 <signal name="SCK">
 <contactref element="R4" pad="1"/>
-<contactref element="PROG_CNT" pad="3"/>
-<wire x1="116.68" y1="63.03" x2="105.62" y2="92.24" width="0" layer="19" extent="1-1"/>
+<contactref element="JP1" pad="7"/>
+<wire x1="-102.27" y1="-46.54" x2="105.62" y2="92.24" width="0" layer="19" extent="1-1"/>
 </signal>
 <signal name="SS_M">
@@
 </signal>
 <signal name="RESET">
-<contactref element="PROG_CNT" pad="5"/>
 <contactref element="U2" pad="20"/>
-<wire x1="90.2932" y1="31.91" x2="119.22" y2="63.03" width="0" layer="19" extent="1-1"/>
+<contactref element="JP1" pad="5"/>
+<wire x1="90.2932" y1="31.91" x2="-102.27" y2="-44" width="0" layer="19" extent="1-1"/>
 </signal>
 <signal name="12V">
