File: hardware/gen4/ControlModule/ControlModule.sch (EAGLE design)
At the start: 0 parts

Commit message: Started working on the microboard
Parts:
- added C1: 1uF, SparkFun-Capacitors:CAP0805
- added C2: 0.01uF, SparkFun-Capacitors:CAP0805
- added C3: 0.1uF, SparkFun-Capacitors:CAP0805
- added FRAME1: FRAME-LETTER, SparkFun-Aesthetics:FRAME-LETTER
- added IC1: XMEGA16A4A, atmel:XMEGA16A4A
- added R1: 10k, SparkFun-Passives:RESISTOR0805-RES
- added R2, R3, R4, R5: 10k, SparkFun-Resistors:RESISTOR0805-RES
- added U$1: 4-POS-DIP, SparkFun-Electromechanical:4-POS-DIP
Connections:
- new net 3.3V: C1.1, C2.1, IC1.VCC, R1.2, U$1.1B, U$1.2B, U$1.3B, U$1.4B
- new net BID0: R2.2, U$1.1A
- new net BID1: R3.2, U$1.2A
- new net BID2: R4.2, U$1.3A
- new net BID3: R5.2, U$1.4A
- new net GND: C1.2, C2.2, C3.1, R2.1, R3.1, R4.1, R5.1
- new net N$1: C3.2, IC1.AVCC, R1.1
