File: hardware/gen4/ControlModule/ControlModule.sch (EAGLE design)
At the start: 39 parts, among them IC1 XMEGA16A4A

Commit message: starting routing
done layout
Parts:
- removed S2: SWITCH-MOMENTARY-2SMD-2, SparkFun-Electromechanical:SWITCH-MOMENTARY-2SMD-2
- added S3: TAC_SWITCHSMD, SparkFun-Retired:TAC_SWITCHSMD
- S1: value SWITCH-MOMENTARY-2SMD-2 -> TAC_SWITCHSMD; device SparkFun-Electromechanical:SWITCH-MOMENTARY-2SMD-2 -> SparkFun-Retired:TAC_SWITCHSMD
Connections:
- net GND: now also S3.2; no longer S2.1
- net RESET: now also S3.4; no longer S2.2
- net XBRST: now also S1.3, S1.4; no longer S1.1
Changed lines of the file:
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@@
 <part name="TX" library="gen3" deviceset="TEST_PT" device=""/>
 <part name="R6" library="SparkFun-Passives" deviceset="RESISTOR" device="0805-RES" value="4.7k"/>
-<part name="S1" library="SparkFun-Electromechanical" deviceset="SWITCH-MOMENTARY-2" device="SMD-2"/>
-<part name="S2" library="SparkFun-Electromechanical" deviceset="SWITCH-MOMENTARY-2" device="SMD-2"/>
 <part name="R7" library="SparkFun-Passives" deviceset="RESISTOR" device="0805-RES" value="10k"/>
 <part name="R8" library="SparkFun-Passives" deviceset="RESISTOR" device="0805-RES" value="80k"/>
@@
 <part name="JP1" library="SparkFun-Connectors" deviceset="M20X2" device="SHROUDED_SMT"/>
 <part name="JP3" library="SparkFun-Connectors" deviceset="M05X2" device="SHD"/>
+<part name="S3" library="SparkFun-Retired" deviceset="TAC_SWITCH" device="SMD" value="TAC_SWITCHSMD"/>
+<part name="S1" library="SparkFun-Retired" deviceset="TAC_SWITCH" device="SMD" value="TAC_SWITCHSMD"/>
 </parts>
 <sheets>
@@
 <instance part="TX" gate="G$1" x="147.32" y="66.04"/>
 <instance part="R6" gate="G$1" x="119.38" y="22.86"/>
-<instance part="S1" gate="G$1" x="132.08" y="27.94" rot="R90"/>
-<instance part="S2" gate="G$1" x="27.94" y="101.6"/>
 <instance part="R7" gate="G$1" x="40.64" y="106.68" rot="R90"/>
 <instance part="R8" gate="G$1" x="127" y="83.82" rot="R90"/>
@@
 <instance part="JP1" gate="G$1" x="30.48" y="154.94"/>
 <instance part="JP3" gate="G$1" x="83.82" y="111.76"/>
+<instance part="S3" gate="S" x="27.94" y="104.14"/>
+<instance part="S1" gate="S" x="134.62" y="27.94" rot="R270"/>
 </instances>
 <busses>
@@
 <wire x1="40.64" y1="101.6" x2="33.02" y2="101.6" width="0.1524" layer="91"/>
 <junction x="40.64" y="101.6"/>
-<pinref part="S2" gate="G$1" pin="2"/>
 <pinref part="R7" gate="G$1" pin="1"/>
+<pinref part="S3" gate="S" pin="4"/>
 </segment>
 <segment>
@@
 </segment>
 <segment>
-<pinref part="S1" gate="G$1" pin="2"/>
 <wire x1="132.08" y1="33.02" x2="132.08" y2="40.64" width="0.1524" layer="91"/>
 <label x="132.08" y="40.64" size="1.778" layer="95" rot="R180"/>
-</segment>
-<segment>
-<pinref part="S2" gate="G$1" pin="1"/>
+<pinref part="S1" gate="S" pin="2"/>
+</segment>
+<segment>
 <wire x1="22.86" y1="101.6" x2="17.78" y2="101.6" width="0.1524" layer="91"/>
 <label x="15.24" y="101.6" size="1.778" layer="95"/>
+<pinref part="S3" gate="S" pin="2"/>
 </segment>
 <segment>
@@
 <segment>
 <pinref part="R6" gate="G$1" pin="2"/>
-<pinref part="S1" gate="G$1" pin="1"/>
 <wire x1="124.46" y1="22.86" x2="132.08" y2="22.86" width="0.1524" layer="91"/>
-<wire x1="132.08" y1="22.86" x2="137.16" y2="22.86" width="0.1524" layer="91"/>
+<wire x1="132.08" y1="22.86" x2="134.62" y2="22.86" width="0.1524" layer="91"/>
+<label x="137.16" y="22.86" size="1.778" layer="95"/>
+<pinref part="S1" gate="S" pin="3"/>
+<wire x1="134.62" y1="22.86" x2="137.16" y2="22.86" width="0.1524" layer="91"/>
+<junction x="134.62" y="22.86"/>
+<pinref part="S1" gate="S" pin="4"/>
 <junction x="132.08" y="22.86"/>
-<label x="137.16" y="22.86" size="1.778" layer="95"/>
-</segment>
-</net>
+</segment>
+</net>

Commit message: routing in progress (comms board)
Connections:
- net GND: now also S1.1, S3.1
- net RESET: now also S3.3
Changed lines of the file:
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@@
 <pinref part="R7" gate="G$1" pin="1"/>
 <pinref part="S3" gate="S" pin="4"/>
+<pinref part="S3" gate="S" pin="3"/>
+<wire x1="33.02" y1="104.14" x2="33.02" y2="101.6" width="0.1524" layer="91"/>
 </segment>
 <segment>
@@
 <label x="132.08" y="40.64" size="1.778" layer="95" rot="R180"/>
 <pinref part="S1" gate="S" pin="2"/>
+<pinref part="S1" gate="S" pin="1"/>
+<wire x1="132.08" y1="33.02" x2="134.62" y2="33.02" width="0.1524" layer="91"/>
 </segment>
 <segment>
@@
 <label x="15.24" y="101.6" size="1.778" layer="95"/>
 <pinref part="S3" gate="S" pin="2"/>
+<pinref part="S3" gate="S" pin="1"/>
+<wire x1="22.86" y1="104.14" x2="22.86" y2="101.6" width="0.1524" layer="91"/>
 </segment>
 <segment>

Commit message: comms board done I think
Parts:
- removed JP3: (no value), SparkFun-Connectors:M05X2SHD
- added JP2: (no value), pinhead:PINHD-2X3
Connections:
- net 3.3V: now also JP2.2; no longer JP3.2
- net DATA: now also JP2.1
- net GND: now also JP2.6; no longer JP3.10, JP3.4, JP3.6, JP3.8
- net MISO: no longer JP3.9
- net MOSI: no longer JP3.1
- net RESET: now also JP2.5; no longer JP3.5
- net SCK: no longer JP3.7
Changed lines of the file:
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@@
 <part name="C6" library="SparkFun-Capacitors" deviceset="CAP" device="0805" value=".01uF"/>
 <part name="JP1" library="SparkFun-Connectors" deviceset="M20X2" device="SHROUDED_SMT"/>
-<part name="JP3" library="SparkFun-Connectors" deviceset="M05X2" device="SHD"/>
 <part name="S3" library="SparkFun-Retired" deviceset="TAC_SWITCH" device="SMD" value="TAC_SWITCHSMD"/>
 <part name="S1" library="SparkFun-Retired" deviceset="TAC_SWITCH" device="SMD" value="TAC_SWITCHSMD"/>
+<part name="JP2" library="pinhead" deviceset="PINHD-2X3" device=""/>
 </parts>
 <sheets>
@@
 <instance part="C6" gate="G$1" x="119.38" y="132.08"/>
 <instance part="JP1" gate="G$1" x="30.48" y="154.94"/>
-<instance part="JP3" gate="G$1" x="83.82" y="111.76"/>
 <instance part="S3" gate="S" x="27.94" y="104.14"/>
 <instance part="S1" gate="S" x="134.62" y="27.94" rot="R270"/>
+<instance part="JP2" gate="A" x="83.82" y="114.3"/>
 </instances>
 <busses>
@@
 <label x="58.42" y="139.7" size="1.778" layer="95" rot="R180"/>
 </segment>
-<segment>
-<wire x1="68.58" y1="106.68" x2="76.2" y2="106.68" width="0.1524" layer="91"/>
-<label x="68.58" y="106.68" size="1.778" layer="95"/>
-<pinref part="JP3" gate="G$1" pin="9"/>
-<junction x="76.2" y="106.68"/>
-</segment>
 </net>
 <net name="MOSI" class="0">
@@
 <label x="58.42" y="142.24" size="1.778" layer="95" rot="R180"/>
 </segment>
-<segment>
-<wire x1="68.58" y1="116.84" x2="76.2" y2="116.84" width="0.1524" layer="91"/>
-<label x="68.58" y="116.84" size="1.778" layer="95"/>
-<pinref part="JP3" gate="G$1" pin="1"/>
-<junction x="76.2" y="116.84"/>
-</segment>
 </net>
 <net name="SCK" class="0">
@@
 <wire x1="53.34" y1="144.78" x2="58.42" y2="144.78" width="0.1524" layer="91"/>
 <label x="58.42" y="144.78" size="1.778" layer="95" rot="R180"/>
-</segment>
-<segment>
-<wire x1="68.58" y1="109.22" x2="76.2" y2="109.22" width="0.1524" layer="91"/>
-<label x="68.58" y="109.22" size="1.778" layer="95"/>
-<pinref part="JP3" gate="G$1" pin="7"/>
-<junction x="76.2" y="109.22"/>
 </segment>
 </net>
@@
 </segment>
 <segment>
-<wire x1="76.2" y1="111.76" x2="68.58" y2="111.76" width="0.1524" layer="91"/>
+<wire x1="81.28" y1="111.76" x2="73.66" y2="111.76" width="0.1524" layer="91"/>
 <label x="68.58" y="111.76" size="1.778" layer="95"/>
-<pinref part="JP3" gate="G$1" pin="5"/>
-<junction x="76.2" y="111.76"/>
+<pinref part="JP2" gate="A" pin="5"/>
+<junction x="81.28" y="111.76"/>
 </segment>
 </net>
@@
 <label x="218.44" y="106.68" size="1.778" layer="95"/>
 <label x="17.78" y="137.16" size="1.778" layer="95"/>
-</segment>
-<segment>
-<wire x1="91.44" y1="111.76" x2="96.52" y2="111.76" width="0.1524" layer="91"/>
-<label x="96.52" y="111.76" size="1.778" layer="95"/>
-<pinref part="JP3" gate="G$1" pin="6"/>
-<junction x="91.44" y="111.76"/>
-<pinref part="JP3" gate="G$1" pin="4"/>
-<wire x1="91.44" y1="114.3" x2="91.44" y2="111.76" width="0.1524" layer="91"/>
-<pinref part="JP3" gate="G$1" pin="8"/>
-<wire x1="91.44" y1="111.76" x2="91.44" y2="109.22" width="0.1524" layer="91"/>
-<pinref part="JP3" gate="G$1" pin="10"/>
-<wire x1="91.44" y1="109.22" x2="91.44" y2="106.68" width="0.1524" layer="91"/>
-<junction x="91.44" y="106.68"/>
-<junction x="91.44" y="109.22"/>
-<junction x="91.44" y="114.3"/>
 </segment>
 <segment>
@@
 <wire x1="22.86" y1="137.16" x2="38.1" y2="137.16" width="0.1524" layer="91"/>
 <wire x1="22.86" y1="137.16" x2="17.78" y2="137.16" width="0.1524" layer="91"/>
+</segment>
+<segment>
+<pinref part="JP2" gate="A" pin="6"/>
+<wire x1="88.9" y1="111.76" x2="96.52" y2="111.76" width="0.1524" layer="91"/>
+<label x="93.98" y="111.76" size="1.778" layer="95"/>
 </segment>
 </net>
@@
 </segment>
 <segment>
-<wire x1="91.44" y1="116.84" x2="96.52" y2="116.84" width="0.1524" layer="91"/>
-<label x="96.52" y="116.84" size="1.778" layer="95"/>
-<pinref part="JP3" gate="G$1" pin="2"/>
-<junction x="91.44" y="116.84"/>
+<wire x1="88.9" y1="116.84" x2="93.98" y2="116.84" width="0.1524" layer="91"/>
+<label x="93.98" y="116.84" size="1.778" layer="95"/>
+<pinref part="JP2" gate="A" pin="2"/>
+<junction x="88.9" y="116.84"/>
 </segment>
 </net>
@@
 <wire x1="48.26" y1="86.36" x2="40.64" y2="86.36" width="0.1524" layer="91"/>
 </segment>
-</net>
+<segment>
+<wire x1="81.28" y1="116.84" x2="73.66" y2="116.84" width="0.1524" layer="91"/>
+<pinref part="JP2" gate="A" pin="1"/>
+<junction x="81.28" y="116.84"/>
+</segment>
+</net>

Commit message: redid debug connector on comms, but clearance checks havent been done
Parts:
- removed JP2: (no value), pinhead:PINHD-2X3
- added JP3: DEBUG, pinhead:PINHD-2X5
Connections:
- net N$1 renamed AVCC
- removed net INT: IC1.PC2
- removed net SCL: IC1.PC1
- removed net SDA: IC1.PC0
- net 3.3V: now also JP3.4; no longer JP2.2
- net DATA: now also JP3.9; no longer JP2.1
- net GND: now also JP3.10; no longer JP2.6
- net RESET: now also JP3.6; no longer JP2.5
Changed lines of the file:
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@@
 <?xml version="1.0" encoding="utf-8"?>
 <!DOCTYPE eagle SYSTEM "eagle.dtd">
-<eagle version="7.2.0">
+<eagle version="7.5.0">
 <drawing>
 <settings>
@@
 <part name="S3" library="SparkFun-Retired" deviceset="TAC_SWITCH" device="SMD" value="TAC_SWITCHSMD"/>
 <part name="S1" library="SparkFun-Retired" deviceset="TAC_SWITCH" device="SMD" value="TAC_SWITCHSMD"/>
-<part name="JP2" library="pinhead" deviceset="PINHD-2X3" device=""/>
+<part name="JP3" library="pinhead" deviceset="PINHD-2X5" device="" value="DEBUG"/>
 </parts>
 <sheets>
@@
 <instance part="S3" gate="S" x="27.94" y="104.14"/>
 <instance part="S1" gate="S" x="134.62" y="27.94" rot="R270"/>
-<instance part="JP2" gate="A" x="83.82" y="114.3"/>
+<instance part="JP3" gate="A" x="83.82" y="109.22"/>
 </instances>
 <busses>
@@
 <pinref part="S3" gate="S" pin="3"/>
 <wire x1="33.02" y1="104.14" x2="33.02" y2="101.6" width="0.1524" layer="91"/>
-</segment>
-<segment>
-<wire x1="81.28" y1="111.76" x2="73.66" y2="111.76" width="0.1524" layer="91"/>
-<label x="68.58" y="111.76" size="1.778" layer="95"/>
-<pinref part="JP2" gate="A" pin="5"/>
-<junction x="81.28" y="111.76"/>
+<junction x="33.02" y="101.6"/>
+</segment>
+<segment>
+<pinref part="JP3" gate="A" pin="6"/>
+<wire x1="88.9" y1="109.22" x2="93.98" y2="109.22" width="0.1524" layer="91"/>
+<label x="93.98" y="109.22" size="1.778" layer="95"/>
 </segment>
 </net>
@@
 <pinref part="S1" gate="S" pin="1"/>
 <wire x1="132.08" y1="33.02" x2="134.62" y2="33.02" width="0.1524" layer="91"/>
+<junction x="132.08" y="33.02"/>
 </segment>
 <segment>
@@
 <pinref part="S3" gate="S" pin="1"/>
 <wire x1="22.86" y1="104.14" x2="22.86" y2="101.6" width="0.1524" layer="91"/>
+<junction x="22.86" y="101.6"/>
 </segment>
 <segment>
@@
 <junction x="218.44" y="114.3"/>
 <label x="218.44" y="106.68" size="1.778" layer="95"/>
-<label x="17.78" y="137.16" size="1.778" layer="95"/>
 </segment>
 <segment>
@@
 <wire x1="22.86" y1="137.16" x2="38.1" y2="137.16" width="0.1524" layer="91"/>
 <wire x1="22.86" y1="137.16" x2="17.78" y2="137.16" width="0.1524" layer="91"/>
-</segment>
-<segment>
-<pinref part="JP2" gate="A" pin="6"/>
-<wire x1="88.9" y1="111.76" x2="96.52" y2="111.76" width="0.1524" layer="91"/>
-<label x="93.98" y="111.76" size="1.778" layer="95"/>
+<label x="15.24" y="137.16" size="1.778" layer="95"/>
+<junction x="22.86" y="137.16"/>
+</segment>
+<segment>
+<pinref part="JP3" gate="A" pin="10"/>
+<wire x1="88.9" y1="104.14" x2="93.98" y2="104.14" width="0.1524" layer="91"/>
+<label x="93.98" y="104.14" size="1.778" layer="95"/>
 </segment>
 </net>
@@
 </segment>
 <segment>
-<wire x1="88.9" y1="116.84" x2="93.98" y2="116.84" width="0.1524" layer="91"/>
-<label x="93.98" y="116.84" size="1.778" layer="95"/>
-<pinref part="JP2" gate="A" pin="2"/>
-<junction x="88.9" y="116.84"/>
-</segment>
-</net>
-<net name="N$1" class="0">
+<pinref part="JP3" gate="A" pin="4"/>
+<wire x1="88.9" y1="111.76" x2="93.98" y2="111.76" width="0.1524" layer="91"/>
+<label x="93.98" y="111.76" size="1.778" layer="95"/>
+</segment>
+</net>
+<net name="AVCC" class="0">
 <segment>
 <pinref part="IC1" gate="G$1" pin="AVCC"/>
@@
 <pinref part="S1" gate="S" pin="4"/>
 <junction x="132.08" y="22.86"/>
-</segment>
-</net>
-<net name="SCL" class="0">
-<segment>
-<wire x1="99.06" y1="40.64" x2="101.6" y2="40.64" width="0.1524" layer="91"/>
-<pinref part="IC1" gate="G$1" pin="PC1"/>
-</segment>
-</net>
-<net name="SDA" class="0">
-<segment>
-<wire x1="99.06" y1="38.1" x2="101.6" y2="38.1" width="0.1524" layer="91"/>
-<pinref part="IC1" gate="G$1" pin="PC0"/>
 </segment>
 </net>
@@
 <wire x1="111.76" y1="137.16" x2="119.38" y2="137.16" width="0.1524" layer="91"/>
 <wire x1="119.38" y1="137.16" x2="119.38" y2="142.24" width="0.1524" layer="91"/>
+<junction x="111.76" y="137.16"/>
+<junction x="119.38" y="137.16"/>
+<junction x="119.38" y="142.24"/>
 </segment>
 <segment>
@@
 <pinref part="C4" gate="G$1" pin="2"/>
 <wire x1="111.76" y1="129.54" x2="104.14" y2="129.54" width="0.1524" layer="91"/>
+<junction x="111.76" y="129.54"/>
+<junction x="119.38" y="129.54"/>
 </segment>
 <segment>
@@
 </segment>
 </net>
-<net name="INT" class="0">
-<segment>
-<wire x1="99.06" y1="43.18" x2="101.6" y2="43.18" width="0.1524" layer="91"/>
-<pinref part="IC1" gate="G$1" pin="PC2"/>
-</segment>
-</net>
 <net name="GLED1" class="0">
 <segment>
@@
 </segment>
 <segment>
-<wire x1="81.28" y1="116.84" x2="73.66" y2="116.84" width="0.1524" layer="91"/>
-<pinref part="JP2" gate="A" pin="1"/>
-<junction x="81.28" y="116.84"/>
-</segment>
-</net>
+<pinref part="JP3" gate="A" pin="9"/>
+<wire x1="81.28" y1="104.14" x2="76.2" y2="104.14" width="0.1524" layer="91"/>
+<label x="76.2" y="104.14" size="1.778" layer="95" rot="MR0"/>
+</segment>
+</net>

Commit message: changed a resistor value
Parts:
- R8: value 80k -> 80.6k
Changed lines of the file:
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@@
 <part name="R6" library="SparkFun-Passives" deviceset="RESISTOR" device="0805-RES" value="4.7k"/>
 <part name="R7" library="SparkFun-Passives" deviceset="RESISTOR" device="0805-RES" value="10k"/>
-<part name="R8" library="SparkFun-Passives" deviceset="RESISTOR" device="0805-RES" value="80k"/>
+<part name="R8" library="SparkFun-Passives" deviceset="RESISTOR" device="0805-RES" value="80.6k"/>
 <part name="R9" library="SparkFun-Passives" deviceset="RESISTOR" device="0805-RES" value="20k"/>
 <part name="C13" library="SparkFun-Capacitors" deviceset="CAP" device="0805" value="1uF"/>
