File: hardware/gen4/MotherBoard/MotherBoard.sch (EAGLE design)
At the start: 0 parts

Commit message: Added power dribbler and batsense to mobo
Parts:
- added 12V, 3.3V: TEST_PT, gen3:TEST_PT
- added 3.3REG: 3.3REG1AREG, gen3:3.3REG1AREG
- added BATCLAMP1, BATCLAMP2: DIODE-ZENERDO214AC, gen3:DIODE-ZENERDO214AC
- added BATT: (no value), con-wago-500:W237-102
- added C10: 47uF, SparkFun-Capacitors:CAP1206
- added C13: 1uF, SparkFun-Capacitors:CAP0805
- added C7: .01uF, SparkFun-Capacitors:CAP0805
- added DRIB: JST-22MM, gen3:JST-22MM
- added DRIB_TRAN: (no value), gen3:N-MOSFETDPAK
- added ON/OFF: SPDT-SWITCH, gen3:SPDT-SWITCH
- added R10: 80k, SparkFun-Passives:RESISTOR0805-RES
- added R16: 20k, SparkFun-Passives:RESISTOR0805-RES
Connections:
- new net 12V: DRIB.P$1, R10.2
- new net 12VGND: 3.3REG.GND, BATT-2.KL, C10.2, C13.2, C7.2, DRIB_TRAN.S
- new net 3.3V: 3.3REG.OUT, 3.3V.P$1, C10.1, C13.1, C7.1
- new net 5V: BATCLAMP1.C
- new net BAT+: BATT-1.KL, ON/OFF.COM, ON/OFF.P1
- new net BATSENSE: BATCLAMP1.A, BATCLAMP2.C, R10.1, R16.2
- new net DRIB: DRIB_TRAN.G
- new net GND: BATCLAMP2.A, R16.1
- new net N$3: 12V.P$1, 3.3REG.IN, ON/OFF.P2
- new net TO_DRIB: DRIB.P$2, DRIB_TRAN.D
Other:
- note added: "15v -> 3v division to measure battery voltage"
- note added: "max gate threshold: 2.6V. should turn on fine with 3.3!"
