File: hardware/gen4/ChargerModule/ChargerModule.sch (EAGLE design)
At the start: 0 parts

Commit message: finished charger module
Parts:
- added C18: 10uF, SparkFun-Capacitors:CAP0805
- added C19: 100pF, SparkFun-Capacitors:CAP0805
- added C20, C21, C23: 47uF, SparkFun-Capacitors:CAP1206
- added CHARGE_D: 1kV, ultrafast, gen3:DIODE-DO214AC
- added CHARGE_U: LT3750, kickerchips:LT3750
- added CONNECTOR: M10SILK_FEMALE_PTH, SparkFun-Connectors:M10SILK_FEMALE_PTH
- added FRAME3: FRAME-LETTER, SparkFun-Aesthetics:FRAME-LETTER
- added R31: 43k, SparkFun-Passives:RESISTOR0805-RES
- added RBG: 2.49k, SparkFun-Passives:RESISTOR0805-RES
- added RSENSE: 10m, SparkFun-Passives:RESISTOR2512
- added RVOUT: 50.4k, SparkFun-Passives:RESISTOR0805-RES
- added SWITCH_Q: (no value), gen3:N-MOSFETDPAK
- added U$1: 32052-TRANSFORMER, gen3:32052-TRANSFORMER
Connections:
- new net 12V: C18.1, C20.1, C21.1, C23.1, CHARGE_U.VCC, CHARGE_U.VT, CONNECTOR.4, CONNECTOR.5, U$1.P$4, U$1.P$5
- new net 12VGND: C20.2, C21.2, C23.2, CONNECTOR.6, CONNECTOR.7, RSENSE.1, U$1.P$10
- new net CAP+: CHARGE_D.C, CONNECTOR.8, CONNECTOR.9
- new net CHARGE: CHARGE_U.CHRG, CONNECTOR.2
- new net DONE: CHARGE_U.~DN, CONNECTOR.1
- new net GND: C18.2, C19.2, CHARGE_U.GND, CONNECTOR.3, RBG.1
- new net N$10: CHARGE_U.RDCM, R31.1
- new net N$24: CHARGE_U.SRC, RSENSE.2, SWITCH_Q.S
- new net N$5: R31.2, RVOUT.2, SWITCH_Q.D, U$1.P$6, U$1.P$7
- new net N$6: C19.1, CHARGE_U.RBG, RBG.2
- new net N$7: CHARGE_U.RV, RVOUT.1
- new net N$9: CHARGE_U.GATE, SWITCH_Q.G
- new net TRANS_OUT: CHARGE_D.A, U$1.P$1
Other:
- note added: "add 100k pullup to 3.3v on micro board, or use internal pullup for done"
