File: hardware/gen4/ChargerModule/ChargerModule.sch (EAGLE design)
At the start: 15 parts

Commit message: added test points
Parts:
- added 12VGND_TEST, CHARGE_TEST, DONE_TEST, DRAIN_TEST, GATE_TEST, GND_TEST: TEST_PT, gen3:TEST_PT
Connections:
- net 12VGND: now also 12VGND_TEST.P$1
- net CHARGE: now also CHARGE_TEST.P$1
- net DONE: now also DONE_TEST.P$1
- net GND: now also GND_TEST.P$1
- net N$5: now also DRAIN_TEST.P$1
- net N$9: now also GATE_TEST.P$1
Other:
- moved on the sheet: RSENSE, SWITCH_Q
Changed lines of the file:
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@@
 <part name="SWITCH_Q" library="gen3" deviceset="N-MOSFET" device="DPAK"/>
 <part name="U$1" library="gen3" deviceset="32052-TRANSFORMER" device=""/>
+<part name="DRAIN_TEST" library="gen3" deviceset="TEST_PT" device=""/>
+<part name="CHARGE_TEST" library="gen3" deviceset="TEST_PT" device=""/>
+<part name="DONE_TEST" library="gen3" deviceset="TEST_PT" device=""/>
+<part name="GATE_TEST" library="gen3" deviceset="TEST_PT" device=""/>
+<part name="GND_TEST" library="gen3" deviceset="TEST_PT" device=""/>
+<part name="12VGND_TEST" library="gen3" deviceset="TEST_PT" device=""/>
 </parts>
 <sheets>
 <sheet>
 <plain>
-<text x="71.12" y="129.54" size="1.778" layer="91">add 100k pullup to 3.3v on
+<text x="15.24" y="124.46" size="1.778" layer="91">add 100k pullup to 3.3v on
 micro board, or use internal
 pullup for done</text>
@@
 <instance part="RVOUT" gate="G$1" x="139.7" y="129.54"/>
 <instance part="RBG" gate="G$1" x="149.86" y="76.2" rot="R90"/>
-<instance part="RSENSE" gate="G$1" x="160.02" y="76.2" rot="R90"/>
+<instance part="RSENSE" gate="G$1" x="162.56" y="76.2" rot="R90"/>
 <instance part="C18" gate="G$1" x="91.44" y="78.74"/>
 <instance part="C19" gate="G$1" x="134.62" y="73.66"/>
@@
 <instance part="CHARGE_D" gate="G$1" x="215.9" y="152.4" rot="R90"/>
 <instance part="C23" gate="G$1" x="198.12" y="73.66"/>
-<instance part="SWITCH_Q" gate="G$1" x="157.48" y="111.76"/>
+<instance part="SWITCH_Q" gate="G$1" x="160.02" y="111.76"/>
 <instance part="U$1" gate="G$1" x="198.12" y="134.62"/>
+<instance part="DRAIN_TEST" gate="G$1" x="162.56" y="124.46"/>
+<instance part="CHARGE_TEST" gate="G$1" x="86.36" y="129.54"/>
+<instance part="DONE_TEST" gate="G$1" x="81.28" y="134.62"/>
+<instance part="GATE_TEST" gate="G$1" x="152.4" y="132.08"/>
+<instance part="GND_TEST" gate="G$1" x="119.38" y="68.58"/>
+<instance part="12VGND_TEST" gate="G$1" x="218.44" y="63.5" rot="R270"/>
 </instances>
 <busses>
@@
 <segment>
 <wire x1="149.86" y1="63.5" x2="134.62" y2="63.5" width="0.1524" layer="91"/>
-<wire x1="134.62" y1="63.5" x2="101.6" y2="63.5" width="0.1524" layer="91"/>
+<wire x1="134.62" y1="63.5" x2="119.38" y2="63.5" width="0.1524" layer="91"/>
+<wire x1="119.38" y1="63.5" x2="101.6" y2="63.5" width="0.1524" layer="91"/>
 <wire x1="101.6" y1="63.5" x2="91.44" y2="63.5" width="0.1524" layer="91"/>
 <wire x1="91.44" y1="76.2" x2="91.44" y2="63.5" width="0.1524" layer="91"/>
@@
 <pinref part="C19" gate="G$1" pin="2"/>
 <pinref part="CHARGE_U" gate="G$1" pin="GND"/>
+<pinref part="GND_TEST" gate="G$1" pin="P$1"/>
+<wire x1="119.38" y1="66.04" x2="119.38" y2="63.5" width="0.1524" layer="91"/>
+<junction x="119.38" y="63.5"/>
 </segment>
 <segment>
@@
 <wire x1="172.72" y1="71.12" x2="172.72" y2="63.5" width="0.1524" layer="91"/>
 <junction x="172.72" y="63.5"/>
-<wire x1="172.72" y1="63.5" x2="160.02" y2="63.5" width="0.1524" layer="91"/>
+<wire x1="172.72" y1="63.5" x2="162.56" y2="63.5" width="0.1524" layer="91"/>
 <pinref part="RSENSE" gate="G$1" pin="1"/>
-<wire x1="160.02" y1="71.12" x2="160.02" y2="63.5" width="0.1524" layer="91"/>
+<wire x1="162.56" y1="71.12" x2="162.56" y2="63.5" width="0.1524" layer="91"/>
 <wire x1="215.9" y1="63.5" x2="198.12" y2="63.5" width="0.1524" layer="91"/>
 <junction x="198.12" y="63.5"/>
 <wire x1="180.34" y1="63.5" x2="180.34" y2="55.88" width="0.1524" layer="91"/>
 <junction x="180.34" y="63.5"/>
+<pinref part="12VGND_TEST" gate="G$1" pin="P$1"/>
+<junction x="215.9" y="63.5"/>
 </segment>
 <segment>
@@
 <net name="N$5" class="0">
 <segment>
-<wire x1="147.32" y1="119.38" x2="160.02" y2="119.38" width="0.1524" layer="91"/>
-<wire x1="160.02" y1="119.38" x2="182.88" y2="119.38" width="0.1524" layer="91"/>
+<wire x1="147.32" y1="119.38" x2="162.56" y2="119.38" width="0.1524" layer="91"/>
+<wire x1="162.56" y1="119.38" x2="182.88" y2="119.38" width="0.1524" layer="91"/>
 <wire x1="182.88" y1="119.38" x2="185.42" y2="119.38" width="0.1524" layer="91"/>
-<wire x1="160.02" y1="116.84" x2="160.02" y2="119.38" width="0.1524" layer="91"/>
-<junction x="160.02" y="119.38"/>
+<wire x1="162.56" y1="116.84" x2="162.56" y2="119.38" width="0.1524" layer="91"/>
+<junction x="162.56" y="119.38"/>
 <wire x1="144.78" y1="114.3" x2="147.32" y2="114.3" width="0.1524" layer="91"/>
 <wire x1="147.32" y1="114.3" x2="147.32" y2="119.38" width="0.1524" layer="91"/>
@@
 <pinref part="U$1" gate="G$1" pin="P$6"/>
 <pinref part="U$1" gate="G$1" pin="P$7"/>
+<pinref part="DRAIN_TEST" gate="G$1" pin="P$1"/>
+<wire x1="162.56" y1="121.92" x2="162.56" y2="119.38" width="0.1524" layer="91"/>
 </segment>
 </net>
@@
 <pinref part="CHARGE_U" gate="G$1" pin="GATE"/>
 <pinref part="SWITCH_Q" gate="G$1" pin="G"/>
+<pinref part="GATE_TEST" gate="G$1" pin="P$1"/>
+<wire x1="152.4" y1="109.22" x2="154.94" y2="109.22" width="0.1524" layer="91"/>
+<wire x1="152.4" y1="129.54" x2="152.4" y2="109.22" width="0.1524" layer="91"/>
+<junction x="152.4" y="109.22"/>
 </segment>
 </net>
@@
 <net name="DONE" class="0">
 <segment>
-<wire x1="101.6" y1="119.38" x2="78.74" y2="119.38" width="0.1524" layer="91"/>
-<label x="78.74" y="119.38" size="1.778" layer="95"/>
+<wire x1="101.6" y1="119.38" x2="81.28" y2="119.38" width="0.1524" layer="91"/>
+<label x="71.12" y="119.38" size="1.778" layer="95"/>
 <pinref part="CHARGE_U" gate="G$1" pin="~DN"/>
+<pinref part="DONE_TEST" gate="G$1" pin="P$1"/>
+<wire x1="81.28" y1="119.38" x2="71.12" y2="119.38" width="0.1524" layer="91"/>
+<wire x1="81.28" y1="132.08" x2="81.28" y2="119.38" width="0.1524" layer="91"/>
+<junction x="81.28" y="119.38"/>
 </segment>
 <segment>
@@
 <net name="CHARGE" class="0">
 <segment>
-<wire x1="101.6" y1="114.3" x2="78.74" y2="114.3" width="0.1524" layer="91"/>
+<wire x1="101.6" y1="114.3" x2="86.36" y2="114.3" width="0.1524" layer="91"/>
 <pinref part="CHARGE_U" gate="G$1" pin="CHRG"/>
-<label x="78.74" y="114.3" size="1.778" layer="95"/>
+<label x="71.12" y="114.3" size="1.778" layer="95"/>
+<pinref part="CHARGE_TEST" gate="G$1" pin="P$1"/>
+<wire x1="86.36" y1="114.3" x2="71.12" y2="114.3" width="0.1524" layer="91"/>
+<wire x1="86.36" y1="127" x2="86.36" y2="114.3" width="0.1524" layer="91"/>
+<junction x="86.36" y="114.3"/>
 </segment>
 <segment>
@@
 <net name="N$24" class="0">
 <segment>
-<wire x1="160.02" y1="106.68" x2="160.02" y2="104.14" width="0.1524" layer="91"/>
-<wire x1="160.02" y1="104.14" x2="160.02" y2="81.28" width="0.1524" layer="91"/>
-<wire x1="132.08" y1="104.14" x2="160.02" y2="104.14" width="0.1524" layer="91"/>
-<junction x="160.02" y="104.14"/>
+<wire x1="162.56" y1="106.68" x2="162.56" y2="104.14" width="0.1524" layer="91"/>
+<wire x1="162.56" y1="104.14" x2="162.56" y2="81.28" width="0.1524" layer="91"/>
+<wire x1="132.08" y1="104.14" x2="162.56" y2="104.14" width="0.1524" layer="91"/>
+<junction x="162.56" y="104.14"/>
 <pinref part="RSENSE" gate="G$1" pin="2"/>
 <pinref part="CHARGE_U" gate="G$1" pin="SRC"/>
