File: hardware/gen6/MotherBoard/KickerBoard.brd (EAGLE design)
At the start: 143.9 x 149.3 mm, 185 parts, among them U1 SAM3S4B

Commit message: new motor controller
Parts:
- removed 5REG3: 3.3REG1AREG, gen3:DPAK
- removed C16, C17, C22, C25, C28, C29, C30, C31, C32: 100nF, SparkFun-Capacitors:0805
- removed C24, C26: 2.2uF, SparkFun-Capacitors:0805
- removed C27: 1nF, SparkFun-Capacitors:0805
- removed FRAME4: FRAME-LETTER, SparkFun-Aesthetics:CREATIVE_COMMONS
- removed FUSE_MOTOR_3, FUSE_MOTOR_5, FUSE_MOTOR_6, FUSE_MOTOR_7: (no value), fuse:TR5
- removed JP1, JP2, JP3, JP4: (no value), SparkFun-Connectors:1X04_SMD_RA_FEMALE
- removed KICKREF: MCP6291T-E/OT, SparkFun-AnalogIC:SOT23-5
- removed MOTOR1, MOTOR2, MOTOR3, MOTOR4: M20X2SHROUDED_SMT, SparkFun-Connectors:2X20_SHROUDED_SMT
- removed R35, R36: 4.7k, SparkFun-Resistors:0805
- removed R38, R40: 1.1M, SparkFun-Passives:0805
- removed R39: 1M, SparkFun-Passives:0805
- removed R41: 5.6k, SparkFun-Passives:0805
- removed R42: 1k, SparkFun-Passives:0805
- removed SV1, SV2: (no value), con-lstb:MA10-1W
- removed U$16: RST-REG, sam3s-lib:SOT23-3
- removed U$20: INDUCTOR, gen3:0805
- removed U1: SAM3S4B, atmel_sam:LQFP64
- added 5REG: 3.3REG1AREG, gen3:DPAK
- added J1, J2, J3, J4: (no value), SparkFun-Connectors:2X5-SHROUDED
- added J5, J6, J7, J8: (no value), SparkFun-Connectors:1X04
- C1: value 10pF -> 1uF; device SparkFun-Capacitors:0805 -> SparkFun-Capacitors:1206
- C10: value 10pF -> .01uF; device SparkFun-Capacitors:0805 -> SparkFun-Capacitors:1206
- R27, R33: value 47k -> 4.7k
- R28, R30: value 47k -> 0
- R32: value 47k -> 200k
- R34: value 10K -> 4.7k
- R37: value 1k -> 100k
- R7: value 1M -> 4.7k; device SparkFun-Passives:0805 -> SparkFun-Resistors:0805
- U$10, U$9: value MOTORCON -> MOTOR_BOARD; device gen3:GEN3CON -> Kicker:MOTOR_BOARD
- U$11: value MOTORCON -> PHEONIX-SCREW-TERM; device gen3:GEN3CON -> SparkFun-Connectors:1X02-PHEONIX
- U$13: value INDUCTOR -> PHEONIX-SCREW-TERM; device gen3:0805 -> SparkFun-Connectors:1X02-PHEONIX
- U$14: value JTA-CONN -> TEENSY_3.5/3.6; device sam3s-lib:JTAG-CONN -> Teensy356:TEENSY_3.5/3.6
- U$15: value 12MHZ-OSC -> XBEE-1B1; device sam3s-lib:CRYSTAL-THRU-12MHZ -> gen3:XBEE-1
- U$8: value MOTORCON -> PCA9306; device gen3:GEN3CON -> SparkFun-AnalogIC:SOIC8
- moved U$11 134.8 mm to (134.6, 70.6), flipped to the top, turned to 270 degrees
- moved U$9 102.2 mm to (39.8, 26.0), flipped to the top, turned to 90 degrees
- moved R28 96.4 mm to (131.7, 93.2), turned to 0 degrees
- moved U$10 95.5 mm to (98.0, 72.9), flipped to the top, turned to 270 degrees
- moved R30 92.9 mm to (131.7, 85.0), turned to 0 degrees
- moved U$13 92.7 mm to (4.09, 33.1), flipped to the top, turned to 90 degrees
- moved C41 84.5 mm to (80.7, 62.4)
- moved C39 81.9 mm to (80.6, 60.4)
- moved C40 80.4 mm to (80.6, 58.5)
- moved U$15 71.0 mm to (124.8, 81.1), turned to 0 degrees
- moved C10 68.4 mm to (120.2, 99.6)
- moved C1 68.2 mm to (117.7, 99.6)
- moved U$8 66.7 mm to (70.8, 48.0), turned to 180 degrees
- moved BB_CON 57.2 mm to (48.0, 8.93)
- moved R19 57.2 mm to (46.0, 12.7)
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- renumbered COMP_LED to KICK_READY
Connections:
- net AND_CHIP renamed CHIP
- net AND_KICK renamed KICK
- removed net N$25: FUSE_MOTOR_7.2, MOTOR4.1, MOTOR4.2, MOTOR4.3, MOTOR4.4, MOTOR4.5, MOTOR4.6
- removed net N$26: FUSE_MOTOR_5.2, MOTOR2.1, MOTOR2.2, MOTOR2.3, MOTOR2.4, MOTOR2.5, MOTOR2.6
- removed net N$27: FUSE_MOTOR_3.2, MOTOR1.1, MOTOR1.2, MOTOR1.3, MOTOR1.4, MOTOR1.5, MOTOR1.6
- removed net N$28: MOTOR3.15, MOTOR3.16, MOTOR3.17, MOTOR3.18, U$9.5, U$9.6
- removed net N$31: C10.1, U$15.P$1, U1.61
- removed net N$37: MOTOR3.11, MOTOR3.12, MOTOR3.13, MOTOR3.14, U$9.3, U$9.4
- removed net N$39: MOTOR1.15, MOTOR1.16, MOTOR1.17, MOTOR1.18, U$11.5, U$11.6
- removed net N$41: KICKREF.3, R38.2, R7.2
- removed net N$42: MOTOR2.20, U$8.8
- removed net N$43: MOTOR2.19, U$8.9
- removed net N$44: MOTOR2.21, U$8.10
- removed net N$45: MOTOR2.23, U$8.11
- removed net N$46: MOTOR2.10, MOTOR2.7, MOTOR2.8, MOTOR2.9, U$8.1, U$8.2
- removed net N$47: MOTOR2.11, MOTOR2.12, MOTOR2.13, MOTOR2.14, U$8.3, U$8.4
- removed net N$48: MOTOR2.15, MOTOR2.16, MOTOR2.17, MOTOR2.18, U$8.5, U$8.6
- removed net N$49: KICKREF.1, R37.1, R40.2
- removed net N$50: MOTOR1.20, U$11.8
- removed net N$51: MOTOR1.19, U$11.9
- removed net N$52: MOTOR1.21, U$11.10
- removed net N$53: MOTOR1.23, U$11.11
- removed net N$54: MOTOR4.15, MOTOR4.16, MOTOR4.17, MOTOR4.18, U$10.5, U$10.6
- removed net N$55: MOTOR4.11, MOTOR4.12, MOTOR4.13, MOTOR4.14, U$10.3, U$10.4
- removed net N$56: MOTOR4.10, MOTOR4.7, MOTOR4.8, MOTOR4.9, U$10.1, U$10.2
- removed net N$57: R39.1, R41.1, R42.2
- removed net N$58: MOTOR3.20, U$9.8
- removed net N$59: MOTOR3.19, U$9.9
- removed net N$60: MOTOR3.21, U$9.10
- removed net N$61: MOTOR3.23, U$9.11
- removed net N$66: MOTOR4.20, U$10.8
- removed net N$67: MOTOR4.19, U$10.9
- removed net N$68: MOTOR4.21, U$10.10
- removed net N$69: MOTOR4.23, U$10.11
- removed net N$70: KICKREF.4, R39.2, R40.1
- removed net N$71: MOTOR1.11, MOTOR1.12, MOTOR1.13, MOTOR1.14, U$11.3, U$11.4
- removed net N$72: MOTOR1.10, MOTOR1.7, MOTOR1.8, MOTOR1.9, U$11.1, U$11.2
- removed net RST: R34.1, U$14.RESET, U$16.1, U1.39
- removed net RST_CTRL: SV1.4
- removed net TCK: R33.1, U$14.RTCK, U$14.TCLK, U1.53
- removed net TDI: R30.1, U$14.TDI
- removed net TDO: R27.1, U$14.TDO, U1.49
- removed net TMS: R28.1, U$14.TMS, U1.51
- removed net TWCK: R36.1, SV1.5, U$17.12, U$21.12, U1.36
- removed net TWD: R35.1, SV1.6, U$17.13, U$21.13, U1.43
- removed net VDDOUT: C26.1, C27.1, C28.2, C29.2, C30.2, C31.2, U1.12, U1.24, U1.54, U1.64, U1.8
- new net CTS: R30.1, U$14.24
- new net RTS: R28.1, U$14.35/A16
- new net RX: U$14.34/A15, U$15.2
- new net SCL: R27.1, U$14.19/A5/SCL, U$8.3
- new net SCL-H: R33.1, U$17.12, U$21.12, U$8.6
- new net SDA: R7.1, U$14.18/A4/SDA, U$8.4
- new net SDA-H: R34.1, U$17.13, U$21.13, U$8.5
- new net TX: U$14.33/A14, U$15.3
- new net XBRST: U$15.5
- net 12V: now also 5REG.GATE, U$11.1, U$13.1; no longer 5REG3.GATE, FUSE_MOTOR_3.1, FUSE_MOTOR_5.1, FUSE_MOTOR_6.1, FUSE_MOTOR_7.1, SV1.10, SV1.8, SV1.9
- net 12VGND: now also U$11.2, U$13.2; no longer MOTOR1.22, MOTOR1.33, MOTOR1.34, MOTOR1.35, MOTOR1.36, MOTOR1.37, MOTOR1.38, MOTOR1.39, MOTOR1.40, MOTOR2.22, MOTOR2.33, MOTOR2.34, MOTOR2.35, MOTOR2.36, MOTOR2.37, MOTOR2.38, MOTOR2.39, MOTOR2.40, MOTOR3.22, MOTOR3.33, MOTOR3.34, MOTOR3.35, MOTOR3.36, MOTOR3.37, MOTOR3.38, MOTOR3.39, MOTOR3.40, MOTOR4.22, MOTOR4.33, MOTOR4.34, MOTOR4.35, MOTOR4.36, MOTOR4.37, MOTOR4.38, MOTOR4.39, MOTOR4.40, R11.2, SV1.1, SV1.2, SV1.3, U$10.7, U$11.7, U$13.1, U$20.1, U$8.7, U$9.7
- net 3.3V: now also C1.2, C10.2, R7.2, U$15.1, U$8.2; no longer C13.2, C16.2, C17.2, C22.1, C24.1, C25.1, C32.2, C35.1, C36.1, C37.1, C38.1, KICKREF.5, R28.2, R30.2, R32.2, R33.2, R34.2, R35.2, R36.2, R41.2, U$14.VCC, U$14.VIN_OPT, U$16.2, U$17.18, U$17.9, U$21.17, U$21.18, U$21.9, U1.1, U1.18, U1.45, U1.58, U1.7
- net 5V: now also 5REG.SOURCE, C35.1, C36.1, C37.1, C38.1, J5.1, J6.1, J7.1, J8.1, R32.2, R33.2, R34.2, U$14.VIN, U$17.18, U$17.9, U$21.17, U$21.18, U$21.9; no longer 5REG3.SOURCE, JP1.4, JP2.4, JP3.4, JP4.4
- net BATSENSE: now also U$14.23/A9; no longer U1.3
- net BB_IN: now also U$14.31/A12; no longer U1.10
- net BB_OUT: now also U$14.32/A13; no longer U1.11
- net BREN0: now also J1.6, U$17.3; no longer MOTOR1.27, U$17.6
- net BREN1: now also J3.6; no longer MOTOR2.27
- net BREN2: now also J4.6; no longer MOTOR3.27
- net BREN3: now also J2.6, U$17.26; no longer MOTOR4.27, U$17.23
- net CHARGE: now also U$14.0/RX; no longer U$17.26
- net CHARGE_DONE: now also U$14.1/TX; no longer U$17.27
- net CHIP_ENABLE: now also U$14.5; no longer U$17.2
- net DIR0: now also J1.8, U$17.2; no longer MOTOR1.25, U$17.5
- net DIR1: now also J3.4, U$21.27; no longer MOTOR2.25, U$21.25
- net DIR2: now also J4.4, U$21.2; no longer MOTOR3.25, U$21.4
- net DIR3: now also J2.8, U$17.27; no longer MOTOR4.25, U$17.24
- net DISCHARGE: now also U$14.4/CANRX; no longer U$17.28
- net DRIB: now also U$14.6; no longer U$17.1
- net ENABLE0: now also J1.4, U$17.4; no longer MOTOR1.30, U$17.7
- net ENABLE1: now also J3.8, U$21.25; no longer MOTOR2.30, U$21.27
- net ENABLE2: now also J4.8, U$21.4; no longer MOTOR3.30, U$21.2
- net ENABLE3: now also J2.4, U$17.25; no longer MOTOR4.30, U$17.22
- net FAULT0: now also J1.2, U$17.5; no longer MOTOR1.31, U$17.8
- net FAULT1: now also J3.10, U$21.24; no longer MOTOR2.31, U$21.28
- net FAULT2: now also J4.10, U$21.5; no longer MOTOR3.31, U$21.1
- net FAULT3: now also J2.2, U$17.24; no longer MOTOR4.31, U$17.21
- net GND: now also 5REG.DRAIN, C10.1, J1.9, J2.9, J3.1, J4.1, J5.3, J6.3, J7.3, J8.3, R11.2, U$14.AGND, U$14.GND, U$15.10, U$8.1; no longer 5REG3.DRAIN, C1.2, C10.2, C16.1, C17.1, C22.2, C24.2, C25.2, C26.2, C27.2, C28.1, C29.1, C30.1, C31.1, C32.1, JP1.2, JP2.2, JP3.2, JP4.2, KICKREF.2, R38.1, R42.1, U$13.2, U$14.GND0, U$14.GND1, U$14.GND3, U$14.GND4, U$14.GND5, U$14.GND6, U$14.GND7, U$14.GND8, U$16.3, U$20.2, U1.17, U1.2, U1.46, U1.60
- net HALLOUT0: now also J1.1; no longer MOTOR1.24
- net HALLOUT1: now also J3.9; no longer MOTOR2.24
- net HALLOUT2: now also J4.9; no longer MOTOR3.24
- net HALLOUT3: now also J2.1; no longer MOTOR4.24
- net INT1: now also U$14.9/CS; no longer U1.16
- net INT2: now also U$14.39/A20; no longer U1.50
- net KICK_ENABLE: now also U$14.7; no longer U$17.3
- net KICK_REF: now also R37.1, U$14.A22/DAC1; no longer R7.1, U1.59
- net LOCKN0: now also J1.10, U$17.1; no longer MOTOR1.26, U$17.4
- net LOCKN1: now also J3.2, U$21.28; no longer MOTOR2.26, U$21.24
- net LOCKN2: now also J4.2, U$21.1; no longer MOTOR3.26, U$21.5
- net LOCKN3: now also J2.10, U$17.28; no longer MOTOR4.26, U$17.25
- net M1QA-1: now also J5.2; no longer JP4.3
- net M1QA-1OUT: now also U$14.27; no longer U1.25
- net M1QA-2: now also J6.2; no longer JP1.3
- net M1QA-2OUT: now also U$14.17/A3; no longer U1.37
- net M1QA-3: now also J7.2; no longer JP2.3
- net M1QA-3OUT: now also U$14.15/A1; no longer U1.42
- net M1QA-4: now also J8.2; no longer JP3.3
- net M1QA-4OUT: now also U$14.25; no longer U1.52
- net M1QB-1: now also J5.4; no longer JP4.1
- net M1QB-1OUT: now also U$14.28; no longer U1.26
- net M1QB-2: now also J6.4; no longer JP1.1
- net M1QB-2OUT: now also U$14.16/A2; no longer U1.38
- net M1QB-3: now also J7.4; no longer JP2.1
- net M1QB-3OUT: now also U$14.14/A0; no longer U1.41
- net M1QB-4: now also J8.4; no longer JP3.1
- net M1QB-4OUT: now also U$14.26; no longer U1.23
- net N$16: now also R30.2, U$15.12; no longer C1.1, U$15.P$2, U1.62
- net N$22: now also C1.1; no longer R32.1, U$14.TRST
- net N$38: now also C13.2, R32.1, U$8.7, U$8.8; no longer MOTOR3.10, MOTOR3.7, MOTOR3.8, MOTOR3.9, U$9.1, U$9.2
- net N$4: now also R28.2, U$15.16; no longer FUSE_MOTOR_6.2, MOTOR3.1, MOTOR3.2, MOTOR3.3, MOTOR3.4, MOTOR3.5, MOTOR3.6
- net PWM0: now also J1.3, U$14.10/CS; no longer MOTOR1.29, U1.48
- net PWM1: now also J3.7, U$14.2; no longer MOTOR2.29, U1.47
- net PWM2: now also J4.7, U$14.3/CANTX; no longer MOTOR3.29, U1.44
- net PWM3: now also J2.3, U$14.29; no longer MOTOR4.29, U1.21
Routing:
- net 12V: track 675.0 -> 36.1 mm, vias 13 -> 10
- net GND: track 551.3 -> 71.6 mm, vias 42 -> 17
- net 3.3V: track 677.3 -> 373.3 mm, vias 24 -> 11
- net 12VGND: track 406.7 -> 181.5 mm, vias 37 -> 15
- net TWD: track 180.3 -> 0.00 mm, vias 15 -> 0
- net CTS: track 0.00 -> 154.9 mm
- net TWCK: track 149.6 -> 0.00 mm, vias 12 -> 0
- net RTS: track 0.00 -> 142.7 mm
- net RX: track 0.00 -> 137.9 mm
- net TX: track 0.00 -> 130.3 mm
- net BB_IN: track 111.1 -> 13.6 mm, vias 8 -> 0
- net FAULT2: track 108.0 -> 11.3 mm, vias 12 -> 0
- net M1QA-3OUT: track 100.7 -> 5.35 mm, vias 3 -> 0
- net M1QA-2OUT: track 94.3 -> 4.89 mm, vias 6 -> 0
- net SCL-H: track 0.00 -> 88.2 mm, vias 0 -> 2
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Other:
- board size 143.9 x 149.3 mm -> 143.9 x 141.8 mm
- board text added: "MOTHERBOARD"

Commit message: started conversion
Parts:
- added IC1: 4011D, 40xx:SO14
- added U1: SN74LVC1G32DCKR, SparkFun-IC-Logic:SOT23-5
- added U2: 74HC1G04, SparkFun-IC-Logic:SOT353
Connections:
- new net N$25: U1.1, U2.2
- new net N$26: IC1.2, U2.4
- new net N$27: IC1.1, U1.2
- new net N$28: U1.4
- new net N$31: IC1.3
- new net VDD: IC1.14
- new net VSS: IC1.7
