File: hardware/gen6/MotherBoard/KickerBoard.brd (EAGLE design)
At the start: 143.9 x 141.8 mm, 155 parts

Commit message: new motor controller2
Parts:
- added R35, R36: 1K, SparkFun-Passives:0805
- added U$16, U$20, U$23, U$24: VNH5019, IAD-Library:MULTIPOWERSO-30
- added U$25: MOSFET-NCH, IAD-Library:TO252-3
Connections:
- new net N$25: R35.1, U$16.5
- new net N$26: R36.1, U$16.9
- net GND: now also U$16.17, U$16.18, U$16.19, U$16.20, U$16.26, U$16.27, U$16.28, U$16.29
