File: hardware/gen6/MotherBoard/KickerBoard.sch (EAGLE design)
At the start: 185 parts, among them U1 SAM3S4B

Commit message: new motor controller
Parts:
- removed 5REG3: 3.3REG1AREG, gen3:3.3REG1AREG
- removed C16, C17, C22, C25, C28, C29, C30, C31, C32: 100nF, SparkFun-Capacitors:CAP0805
- removed C24, C26: 2.2uF, SparkFun-Capacitors:CAP0805
- removed C27: 1nF, SparkFun-Capacitors:CAP0805
- removed COMP_LED: (no value), SparkFun-LED:LED1206
- removed FRAME4: FRAME-LETTER, SparkFun-Aesthetics:FRAME-LETTER
- removed FUSE_MOTOR_3, FUSE_MOTOR_5, FUSE_MOTOR_6, FUSE_MOTOR_7: (no value), fuse:TR5
- removed JP1, JP2, JP3, JP4: (no value), SparkFun-Connectors:M04SMD_RA_FEMALE
- removed KICKREF: MCP6291T-E/OT, SparkFun-AnalogIC:MCP6291T-E/OT
- removed MOTOR1, MOTOR2, MOTOR3, MOTOR4: M20X2SHROUDED_SMT, SparkFun-Connectors:M20X2SHROUDED_SMT
- removed R35, R36: 4.7k, SparkFun-Resistors:RESISTOR0805-RES
- removed R38, R40: 1.1M, SparkFun-Passives:RESISTOR0805-RES
- removed R39: 1M, SparkFun-Passives:RESISTOR0805-RES
- removed R41: 5.6k, SparkFun-Passives:RESISTOR0805-RES
- removed R42: 1k, SparkFun-Passives:RESISTOR0805-RES
- removed SV1, SV2: (no value), con-lstb:MA10-1W
- removed U$16: RST-REG, sam3s-lib:RST-REG
- removed U$20: INDUCTOR, gen3:INDUCTOR
- removed U1: SAM3S4B, atmel_sam:SAM3S4B
- added 5REG: 3.3REG1AREG, gen3:3.3REG1AREG
- added J1, J2, J3, J4: (no value), SparkFun-Connectors:M05X2SHD
- added J5, J6, J7, J8: (no value), SparkFun-Connectors:M04PTH
- added KICK_READY: (no value), SparkFun-LED:LED1206
- C1: value 10pF -> 1uF; device SparkFun-Capacitors:CAP0805 -> SparkFun-Capacitors:CAP1206
- C10: value 10pF -> .01uF; device SparkFun-Capacitors:CAP0805 -> SparkFun-Capacitors:CAP1206
- R27, R33: value 47k -> 4.7k
- R28, R30: value 47k -> 0
- R32: value 47k -> 200k
- R34: value 10K -> 4.7k
- R37: value 1k -> 100k
- R7: value 1M -> 4.7k; device SparkFun-Passives:RESISTOR0805-RES -> SparkFun-Resistors:RESISTOR0805-RES
- U$10, U$9: value MOTORCON -> MOTOR_BOARD; device gen3:MOTORCON -> Kicker:MOTOR_BOARD
- U$11: value MOTORCON -> PHEONIX-SCREW-TERM; device gen3:MOTORCON -> SparkFun-Connectors:PHEONIX-SCREW-TERM
- U$13: value INDUCTOR -> PHEONIX-SCREW-TERM; device gen3:INDUCTOR -> SparkFun-Connectors:PHEONIX-SCREW-TERM
- U$14: value JTA-CONN -> TEENSY_3.5/3.6; device sam3s-lib:JTA-CONN -> Teensy356:TEENSY_3.5/3.6
- U$15: value 12MHZ-OSC -> XBEE-1B1; device sam3s-lib:12MHZ-OSC -> gen3:XBEE-1B1
- U$8: value MOTORCON -> PCA9306; device gen3:MOTORCON -> SparkFun-AnalogIC:PCA9306
Connections:
- net AND_CHIP renamed CHIP
- net AND_KICK renamed KICK
- removed net N$25: FUSE_MOTOR_7.2, MOTOR4.1, MOTOR4.2, MOTOR4.3, MOTOR4.4, MOTOR4.5, MOTOR4.6
- removed net N$26: FUSE_MOTOR_5.2, MOTOR2.1, MOTOR2.2, MOTOR2.3, MOTOR2.4, MOTOR2.5, MOTOR2.6
- removed net N$27: FUSE_MOTOR_3.2, MOTOR1.1, MOTOR1.2, MOTOR1.3, MOTOR1.4, MOTOR1.5, MOTOR1.6
- removed net N$28: MOTOR3.15, MOTOR3.16, MOTOR3.17, MOTOR3.18, U$9.P$6, U$9.P$7
- removed net N$31: C10.1, U$15.P$1, U1.XOUT/PB8
- removed net N$37: MOTOR3.11, MOTOR3.12, MOTOR3.13, MOTOR3.14, U$9.P$8, U$9.P$9
- removed net N$39: MOTOR1.15, MOTOR1.16, MOTOR1.17, MOTOR1.18, U$11.P$6, U$11.P$7
- removed net N$41: KICKREF.+IN, R38.2, R7.2
- removed net N$42: MOTOR2.20, U$8.P$4
- removed net N$43: MOTOR2.19, U$8.P$3
- removed net N$44: MOTOR2.21, U$8.P$2
- removed net N$45: MOTOR2.23, U$8.P$1
- removed net N$46: MOTOR2.10, MOTOR2.7, MOTOR2.8, MOTOR2.9, U$8.P$10, U$8.P$11
- removed net N$47: MOTOR2.11, MOTOR2.12, MOTOR2.13, MOTOR2.14, U$8.P$8, U$8.P$9
- removed net N$48: MOTOR2.15, MOTOR2.16, MOTOR2.17, MOTOR2.18, U$8.P$6, U$8.P$7
- removed net N$49: KICKREF.OUT, R37.1, R40.2
- removed net N$50: MOTOR1.20, U$11.P$4
- removed net N$51: MOTOR1.19, U$11.P$3
- removed net N$52: MOTOR1.21, U$11.P$2
- removed net N$53: MOTOR1.23, U$11.P$1
- removed net N$54: MOTOR4.15, MOTOR4.16, MOTOR4.17, MOTOR4.18, U$10.P$6, U$10.P$7
- removed net N$55: MOTOR4.11, MOTOR4.12, MOTOR4.13, MOTOR4.14, U$10.P$8, U$10.P$9
- removed net N$56: MOTOR4.10, MOTOR4.7, MOTOR4.8, MOTOR4.9, U$10.P$10, U$10.P$11
- removed net N$57: R39.1, R41.1, R42.2
- removed net N$58: MOTOR3.20, U$9.P$4
- removed net N$59: MOTOR3.19, U$9.P$3
- removed net N$60: MOTOR3.21, U$9.P$2
- removed net N$61: MOTOR3.23, U$9.P$1
- removed net N$66: MOTOR4.20, U$10.P$4
- removed net N$67: MOTOR4.19, U$10.P$3
- removed net N$68: MOTOR4.21, U$10.P$2
- removed net N$69: MOTOR4.23, U$10.P$1
- removed net N$70: KICKREF.-IN, R39.2, R40.1
- removed net N$71: MOTOR1.11, MOTOR1.12, MOTOR1.13, MOTOR1.14, U$11.P$8, U$11.P$9
- removed net N$72: MOTOR1.10, MOTOR1.7, MOTOR1.8, MOTOR1.9, U$11.P$10, U$11.P$11
- removed net RST: R34.1, U$14.RESET, U$16./RST, U1.NRST
- removed net RST_CTRL: SV1.4
- removed net TCK: R33.1, U$14.RTCK, U$14.TCLK, U1.TCK/SWCLK/PB7
- removed net TDI: R30.1, U$14.TDI
- removed net TDO: R27.1, U$14.TDO, U1.TDO/PB5
- removed net TMS: R28.1, U$14.TMS, U1.TMS/SWDIO/PB6
- removed net TWCK: R36.1, SV1.5, U$17.SCK, U$21.SCK, U1.PA4
- removed net TWD: R35.1, SV1.6, U$17.SDA, U$21.SDA, U1.PA3
- removed net VDDOUT: C26.1, C27.1, C28.2, C29.2, C30.2, C31.2, U1.VDDCORE, U1.VDDCORE@1, U1.VDDCORE@2, U1.VDDOUT, U1.VDDPLL
- new net CTS: R30.1, U$14.24
- new net RTS: R28.1, U$14.35/A16
- new net RX: U$14.34/A15, U$15.DOUT
- new net SCL: R27.1, U$14.19/A5/SCL, U$8.SCL1
- new net SCL-H: R33.1, U$17.SCK, U$21.SCK, U$8.SCL2
- new net SDA: R7.1, U$14.18/A4/SDA, U$8.SDA1
- new net SDA-H: R34.1, U$17.SDA, U$21.SDA, U$8.SDA2
- new net TX: U$14.33/A14, U$15.DIN
- new net XBRST: U$15.RESET
- net 12V: now also 5REG.IN, U$11.1, U$13.1; no longer 5REG3.IN, FUSE_MOTOR_3.1, FUSE_MOTOR_5.1, FUSE_MOTOR_6.1, FUSE_MOTOR_7.1, SV1.10, SV1.8, SV1.9
- net 12VGND: now also U$11.2, U$13.2; no longer MOTOR1.22, MOTOR1.33, MOTOR1.34, MOTOR1.35, MOTOR1.36, MOTOR1.37, MOTOR1.38, MOTOR1.39, MOTOR1.40, MOTOR2.22, MOTOR2.33, MOTOR2.34, MOTOR2.35, MOTOR2.36, MOTOR2.37, MOTOR2.38, MOTOR2.39, MOTOR2.40, MOTOR3.22, MOTOR3.33, MOTOR3.34, MOTOR3.35, MOTOR3.36, MOTOR3.37, MOTOR3.38, MOTOR3.39, MOTOR3.40, MOTOR4.22, MOTOR4.33, MOTOR4.34, MOTOR4.35, MOTOR4.36, MOTOR4.37, MOTOR4.38, MOTOR4.39, MOTOR4.40, R11.2, SV1.1, SV1.2, SV1.3, U$10.P$5, U$11.P$5, U$13.P$1, U$20.P$1, U$8.P$5, U$9.P$5
- net 3.3V: now also C1.2, C10.2, KICK_READY.A, R7.2, U$15.VDD, U$8.VREF1; no longer C13.2, C16.2, C17.2, C22.1, C24.1, C25.1, C32.2, C35.1, C36.1, C37.1, C38.1, COMP_LED.A, KICKREF.V+, R28.2, R30.2, R32.2, R33.2, R34.2, R35.2, R36.2, R41.2, U$14.VIN, U$14.VIN_OPT, U$16.VDD, U$17.RESET/, U$17.VDD, U$21.A2, U$21.RESET/, U$21.VDD, U1.ADVREF, U1.VDDIN, U1.VDDIO, U1.VDDIO@1, U1.VDDIO@2
- net 5V: now also 5REG.OUT, C35.1, C36.1, C37.1, C38.1, J5.1, J6.1, J7.1, J8.1, R32.2, R33.2, R34.2, U$14.VIN, U$17.RESET/, U$17.VDD, U$21.A2, U$21.RESET/, U$21.VDD; no longer 5REG3.OUT, JP1.4, JP2.4, JP3.4, JP4.4
- net BATSENSE: now also U$14.23/A9; no longer U1.PB0/AD4
- net BB_IN: now also U$14.31/A12; no longer U1.PA18/AD1
- net BB_OUT: now also U$14.32/A13; no longer U1.PA21/AD8
- net BREN0: now also J1.6, U$17.GPB2; no longer MOTOR1.27, U$17.GPB5
- net BREN1: now also J3.6; no longer MOTOR2.27
- net BREN2: now also J4.6; no longer MOTOR3.27
- net BREN3: now also J2.6, U$17.GPA5; no longer MOTOR4.27, U$17.GPA2
- net CHARGE: now also U$14.0/RX; no longer U$17.GPA5
- net CHARGE_DONE: now also U$14.1/TX; no longer U$17.GPA6
- net CHIP_ENABLE: now also U$14.5; no longer U$17.GPB1
- net DIR0: now also J1.8, U$17.GPB1; no longer MOTOR1.25, U$17.GPB4
- net DIR1: now also J3.4, U$21.GPA6; no longer MOTOR2.25, U$21.GPA4
- net DIR2: now also J4.4, U$21.GPB1; no longer MOTOR3.25, U$21.GPB3
- net DIR3: now also J2.8, U$17.GPA6; no longer MOTOR4.25, U$17.GPA3
- net DISCHARGE: now also U$14.4/CANRX; no longer U$17.GPA7
- net DRIB: now also U$14.6; no longer U$17.GPB0
- net ENABLE0: now also J1.4, U$17.GPB3; no longer MOTOR1.30, U$17.GPB6
- net ENABLE1: now also J3.8, U$21.GPA4; no longer MOTOR2.30, U$21.GPA6
- net ENABLE2: now also J4.8, U$21.GPB3; no longer MOTOR3.30, U$21.GPB1
- net ENABLE3: now also J2.4, U$17.GPA4; no longer MOTOR4.30, U$17.GPA1
- net FAULT0: now also J1.2, U$17.GPB4; no longer MOTOR1.31, U$17.GPB7
- net FAULT1: now also J3.10, U$21.GPA3; no longer MOTOR2.31, U$21.GPA7
- net FAULT2: now also J4.10, U$21.GPB4; no longer MOTOR3.31, U$21.GPB0
- net FAULT3: now also J2.2, U$17.GPA3; no longer MOTOR4.31, U$17.GPA0
- net GND: now also 5REG.GND, C10.1, J1.9, J2.9, J3.1, J4.1, J5.3, J6.3, J7.3, J8.3, R11.2, U$14.AGND, U$14.GND, U$15.GND, U$8.GND; no longer 5REG3.GND, C1.2, C10.2, C16.1, C17.1, C22.2, C24.2, C25.2, C26.2, C27.2, C28.1, C29.1, C30.1, C31.1, C32.1, JP1.2, JP2.2, JP3.2, JP4.2, KICKREF.V-, R38.1, R42.1, U$13.P$2, U$14.GND0, U$14.GND1, U$14.GND3, U$14.GND4, U$14.GND5, U$14.GND6, U$14.GND7, U$14.GND8, U$16.VSS, U$20.P$2, U1.GND, U1.GND@1, U1.GND@2, U1.GND@3
- net HALLOUT0: now also J1.1; no longer MOTOR1.24
- net HALLOUT1: now also J3.9; no longer MOTOR2.24
- net HALLOUT2: now also J4.9; no longer MOTOR3.24
- net HALLOUT3: now also J2.1; no longer MOTOR4.24
- net INT1: now also U$14.9/CS; no longer U1.PA20/AD3
- net INT2: now also U$14.39/A20; no longer U1.JTAGSEL
- net KICK_ENABLE: now also U$14.7; no longer U$17.GPB2
- net KICK_REF: now also R37.1, U$14.A22/DAC1; no longer R7.1, U1.PB13/DAC0
- net LOCKN0: now also J1.10, U$17.GPB0; no longer MOTOR1.26, U$17.GPB3
- net LOCKN1: now also J3.2, U$21.GPA7; no longer MOTOR2.26, U$21.GPA3
- net LOCKN2: now also J4.2, U$21.GPB0; no longer MOTOR3.26, U$21.GPB4
- net LOCKN3: now also J2.10, U$17.GPA7; no longer MOTOR4.26, U$17.GPA4
- net M1QA-1: now also J5.2; no longer JP4.3
- net M1QA-1OUT: now also U$14.27; no longer U1.PA25
- net M1QA-2: now also J6.2; no longer JP1.3
- net M1QA-2OUT: now also U$14.17/A3; no longer U1.PA27
- net M1QA-3: now also J7.2; no longer JP2.3
- net M1QA-3OUT: now also U$14.15/A1; no longer U1.PA30
- net M1QA-4: now also J8.2; no longer JP3.3
- net M1QA-4OUT: now also U$14.25; no longer U1.PA31
- net M1QB-1: now also J5.4; no longer JP4.1
- net M1QB-1OUT: now also U$14.28; no longer U1.PA26
- net M1QB-2: now also J6.4; no longer JP1.1
- net M1QB-2OUT: now also U$14.16/A2; no longer U1.PA28
- net M1QB-3: now also J7.4; no longer JP2.1
- net M1QB-3OUT: now also U$14.14/A0; no longer U1.PA29
- net M1QB-4: now also J8.4; no longer JP3.1
- net M1QB-4OUT: now also U$14.26; no longer U1.PA24
- net N$16: now also R30.2, U$15.CTS; no longer C1.1, U$15.P$2, U1.XIN/PB9
- net N$22: now also C1.1; no longer R32.1, U$14.TRST
- net N$33: now also KICK_READY.C; no longer COMP_LED.C
- net N$38: now also C13.2, R32.1, U$8.EN, U$8.VREF2; no longer MOTOR3.10, MOTOR3.7, MOTOR3.8, MOTOR3.9, U$9.P$10, U$9.P$11
- net N$4: now also R28.2, U$15.RTS; no longer FUSE_MOTOR_6.2, MOTOR3.1, MOTOR3.2, MOTOR3.3, MOTOR3.4, MOTOR3.5, MOTOR3.6
- net PWM0: now also J1.3, U$14.10/CS; no longer MOTOR1.29, U1.PA0
- net PWM1: now also J3.7, U$14.2; no longer MOTOR2.29, U1.PA1
- net PWM2: now also J4.7, U$14.3/CANTX; no longer MOTOR3.29, U1.PA2
- net PWM3: now also J2.3, U$14.29; no longer MOTOR4.29, U1.PA14
Other:
- note added: "Consider whether or not we should use the on-board 3.3V regulator"
- note added: "MOTOR0"
- note added: "MOTOR1"
- note added: "MOTOR2"
- note added: "MOTOR3"
- note removed: "Differential Amplifier: Needed since the DAC on the MCU has a minimum output voltage of ~0.5V, but we want KICK_REF to range from approximately 0 to 2.5 V"
- note removed: "P8, P9, P10 are for Hall Sensors outputs... needed for proper operation of motor controller"
- note removed: "There are 8 Quad Encoder Signals (MXQY) where X refers to the motor number (0-3) and Y referse to the signal (A or B)."
- note removed: "Voff"
- moved on the sheet: 12V, 3.3REG1, 3.3V, BAT, BATCLAMP2, BATT-1, BATT-2, BB_CON, C1, C10, C11, C12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

Commit message: new motor controller2
Parts:
- added R35, R36: 1K, SparkFun-Passives:RESISTOR0805-RES
- added U$16, U$20, U$23, U$24: VNH5019, IAD-Library:VNH5019
- added U$25: MOSFET-NCH, IAD-Library:MOSFET-NCH
Connections:
- new net N$25: R35.1, U$16.ENA/DIAGA
- new net N$26: R36.1, U$16.ENB/DIAGB
- net GND: now also U$16.GNDA, U$16.GNDB
