File: hardware/gen6/MotorModule/MotorBoard.sch (EAGLE design)
At the start: 63 parts, among them IC1 4011D, Q7 PSMN013-30MLC, U1 SN74LVC1G32DCKR, U2 74HC1G04

Commit message: oh dear lord
Parts:
- added U$3: VNH5019A-E, new-st:VNH5019A-E
- Q7: value PSMN013-30MLC -> IRFP250; device transistor-power:PSMN013-30MLC -> transistor-power:IRFP250
Connections:
- new net N$3: Q7.G, U$3.CP
- net +5V: now also U$3.VBAT
- net GND: now also U$3.GNDA, U$3.GNDB
- net N$23: now also U$3.ENA/DIAGA, U$3.ENB/DIAGB
- net N$24: now also U$3.INA
- net N$30: now also U$3.INB
- net N$32: now also U$3.PWM
- net N$34: now also U$3.CS
- net N$36: now also U$3.VCC
- net N$37: now also U$3.OUTB
- net N$39: now also U$3.OUTA
Changed lines of the file:
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@@
 <part name="SUPPLY3" library="supply2" library_urn="urn:adsk.eagle:library:372" deviceset="GND" device=""/>
 <part name="P+3" library="supply1" library_urn="urn:adsk.eagle:library:371" deviceset="+5V" device="" value="VDD"/>
-<part name="Q7" library="transistor-power" library_urn="urn:adsk.eagle:library:400" deviceset="PSMN013-30MLC" device="" package3d_urn="urn:adsk.eagle:package:29530/1"/>
+<part name="U$3" library="new-st" deviceset="VNH5019A-E" device="" package3d_urn="urn:adsk.eagle:package:26846/1"/>
+<part name="Q7" library="transistor-power" library_urn="urn:adsk.eagle:library:400" deviceset="IRFP25*" device="" package3d_urn="urn:adsk.eagle:package:29508/1" technology="0"/>
 </parts>
 <sheets>
@@
 <attribute name="VALUE" x="421.64" y="7.62" size="1.778" layer="96" rot="R90"/>
 </instance>
+<instance part="U$3" gate="VNH5019A-E" x="469.9" y="-35.56" smashed="yes"/>
 <instance part="Q7" gate="G$1" x="485.14" y="7.62" smashed="yes" rot="MR90">
 <attribute name="NAME" x="487.68" y="13.97" size="1.778" layer="95" rot="MR90"/>
@@
 <junction x="441.96" y="-58.42"/>
 <pinref part="SUPPLY3" gate="GND" pin="GND"/>
+<pinref part="U$3" gate="VNH5019A-E" pin="GNDA"/>
+<pinref part="U$3" gate="VNH5019A-E" pin="GNDB"/>
 </segment>
 </net>
@@
 <pinref part="R19" gate="G$1" pin="1"/>
 <wire x1="447.04" y1="-17.78" x2="436.88" y2="-17.78" width="0.1524" layer="91"/>
+<pinref part="U$3" gate="VNH5019A-E" pin="INA"/>
 </segment>
 </net>
@@
 <pinref part="R21" gate="G$1" pin="1"/>
 <wire x1="447.04" y1="-22.86" x2="431.8" y2="-22.86" width="0.1524" layer="91"/>
+<pinref part="U$3" gate="VNH5019A-E" pin="INB"/>
 </segment>
 </net>
@@
 <pinref part="R20" gate="G$1" pin="1"/>
 <wire x1="447.04" y1="-30.48" x2="434.34" y2="-30.48" width="0.1524" layer="91"/>
+<pinref part="U$3" gate="VNH5019A-E" pin="PWM"/>
 </segment>
 </net>
@@
 <junction x="434.34" y="-43.18"/>
 <wire x1="447.04" y1="-43.18" x2="434.34" y2="-43.18" width="0.1524" layer="91"/>
+<pinref part="U$3" gate="VNH5019A-E" pin="CS"/>
 </segment>
 </net>
@@
 <wire x1="495.3" y1="-68.58" x2="495.3" y2="-53.34" width="0.1524" layer="91"/>
 <junction x="535.94" y="-68.58"/>
+<pinref part="U$3" gate="VNH5019A-E" pin="OUTB"/>
 </segment>
 </net>
@@
 <junction x="535.94" y="-35.56"/>
 <wire x1="495.3" y1="-35.56" x2="535.94" y2="-35.56" width="0.1524" layer="91"/>
+<pinref part="U$3" gate="VNH5019A-E" pin="OUTA"/>
 </segment>
 </net>
@@
 <wire x1="505.46" y1="-25.4" x2="505.46" y2="10.16" width="0.1524" layer="91"/>
 <junction x="505.46" y="10.16"/>
+<pinref part="U$3" gate="VNH5019A-E" pin="VCC"/>
 <pinref part="Q7" gate="G$1" pin="D"/>
 </segment>
@@
 <wire x1="472.44" y1="10.16" x2="472.44" y2="5.08" width="0.1524" layer="91"/>
 <wire x1="472.44" y1="10.16" x2="480.06" y2="10.16" width="0.1524" layer="91"/>
+<pinref part="U$3" gate="VNH5019A-E" pin="VBAT"/>
 <pinref part="Q7" gate="G$1" pin="S"/>
 </segment>
@@
 <wire x1="444.5" y1="-10.16" x2="444.5" y2="-5.08" width="0.1524" layer="91"/>
 <junction x="444.5" y="-5.08"/>
-</segment>
-</net>
+<pinref part="U$3" gate="VNH5019A-E" pin="ENA/DIAGA"/>
+<pinref part="U$3" gate="VNH5019A-E" pin="ENB/DIAGB"/>
+</segment>
+</net>
+<net name="N$3" class="0">
+<segment>
+<pinref part="U$3" gate="VNH5019A-E" pin="CP"/>
+<pinref part="Q7" gate="G$1" pin="G"/>
+</segment>
+</net>
