File: hardware/gen5/MotherBoard/KickerBoard-new.brd (EAGLE design)
At the start: 143.9 x 141.8 mm, 226 parts

Commit message: almost done2
Parts:
- moved BB_CON 50.2 mm to (96.4, 22.3)
- moved C12 50.2 mm to (96.4, 26.0)
- moved R19 50.2 mm to (94.4, 26.0)
- moved R20 50.2 mm to (100.3, 25.9)
- moved U$19 10.9 mm to (67.5, 28.5)
- moved GND 8.21 mm to (81.6, 19.7)
- moved 3.3V 5.81 mm to (78.6, 19.8)
- moved C43 0.71 mm to (113.4, 49.4)
- moved C44 0.71 mm to (114.0, 47.5)
- moved C28 0.53 mm to (35.7, 34.1)
- moved ON/OFF 0.53 mm to (130.1, 53.1)
- moved R74 0.18 mm to (35.7, 32.5)
Connections:
- removed net N$22: C1.1
- net GND: now also C1.1
Routing:
- net 5V: track 82.7 -> 353.7 mm, vias 3 -> 20
- net INB_3: track 0.00 -> 53.1 mm, vias 0 -> 2
- net 3.3V: track 266.5 -> 307.6 mm, vias 12 -> 14
- net GND: track 69.8 -> 103.2 mm, vias 17 -> 28
- net 12V: track 129.0 -> 151.7 mm, vias 16 -> 18
- net BB_OUT: track 0.00 -> 13.9 mm, vias 0 -> 1
- net N$42: track 35.7 -> 47.2 mm
- net BB_IN: track 0.00 -> 10.4 mm
- net OUTA_2: track 31.7 -> 40.7 mm
- net OUTB_1: track 47.9 -> 56.8 mm
- net OUTB_2: track 50.9 -> 58.9 mm
- net OUTA_3: track 35.8 -> 40.0 mm
- net N$1: track 8.22 -> 4.33 mm
- net 12VGND: track 263.4 -> 266.7 mm, vias 28 -> 29
- net N$50: track 0.00 -> 2.92 mm
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
Commit message: almost done3
Routing:
- net 12VGND: track 266.7 -> 232.3 mm
- net INB_3: track 53.1 -> 51.9 mm
- net CS_3: track 19.7 -> 19.3 mm, vias 2 -> 1
- net DISCHARGE: track 94.4 -> 94.8 mm, vias 4 -> 6
- net ENB_3: track 53.6 -> 54.0 mm, vias 3 -> 5

Commit message: clean up and bom
Parts:
- removed KICK_Q, KICK_Q1: (no value), gen3:DPAK
- removed U$10, U$9: MOTOR_BOARD, Kicker:MOTOR_BOARD
- added Q1, Q2: IXFT94N30P3, transistor-power:TO268
- moved R2 10.2 mm to (29.6, 101.3)
- moved R1 9.11 mm to (30.8, 75.9)
- moved R21 8.14 mm to (124.8, 110.8), turned to 180 degrees
- moved C24 6.78 mm to (28.4, 60.8)
- moved C17 6.29 mm to (28.8, 63.3)
- moved U$20 6.06 mm to (25.8, 56.4)
- moved PW_LED1 5.76 mm to (124.6, 113.3), turned to 180 degrees
- moved R11 4.82 mm to (32.4, 88.0), turned to 270 degrees
- moved CAP+_TEST 4.50 mm to (32.8, 98.6)
- moved C16 2.32 mm to (16.9, 62.4)
Connections:
- net 12VGND: now also Q1.E, Q2.E; no longer KICK_Q.SOURCE, KICK_Q1.SOURCE
- net LOWCHIP: now also Q2.C@1, Q2.C@2; no longer KICK_Q1.DRAIN
- net LOWKICK: now also Q1.C@1, Q1.C@2; no longer KICK_Q.DRAIN
- net N$3: now also Q2.G; no longer KICK_Q1.GATE
- net N$8: now also Q1.G; no longer KICK_Q.GATE
Routing:
- net 12V: track 151.7 -> 170.5 mm, vias 18 -> 17
- net GND: track 103.5 -> 121.7 mm
- net N$42: track 47.2 -> 61.2 mm, vias 4 -> 6
- net CAP+: track 201.5 -> 214.4 mm
- net N$5: track 52.9 -> 62.4 mm
- net N$2: track 61.0 -> 52.1 mm
- net N$41: track 21.3 -> 29.9 mm
- net 12VGND: track 232.3 -> 236.9 mm, vias 29 -> 41
- net LOWKICK: track 18.0 -> 20.8 mm
- net LOWCHIP: track 19.1 -> 21.1 mm
- net M1QA-1OUT: track 72.2 -> 73.6 mm
- net N$20: track 3.17 -> 1.81 mm
- net M1QB-1OUT: track 72.1 -> 73.4 mm
- net DISCHARGE: track 94.8 -> 95.6 mm
- net N$3: track 2.64 -> 3.46 mm
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