File: hardware/gen5/MotherBoard/KickerBoard-new.sch (EAGLE design)
At the start: 226 parts

Commit message: almost done2
Connections:
- removed net N$22: C1.1
- net GND: now also C1.1
Changed lines of the file:
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@@
 <pinref part="C10" gate="G$1" pin="1"/>
 <wire x1="403.86" y1="86.36" x2="403.86" y2="91.44" width="0.1524" layer="91"/>
-<wire x1="403.86" y1="91.44" x2="383.54" y2="91.44" width="0.1524" layer="91"/>
+<wire x1="403.86" y1="91.44" x2="393.7" y2="91.44" width="0.1524" layer="91"/>
+<wire x1="393.7" y1="91.44" x2="383.54" y2="91.44" width="0.1524" layer="91"/>
 <wire x1="383.54" y1="91.44" x2="383.54" y2="88.9" width="0.1524" layer="91"/>
 <label x="375.92" y="88.9" size="1.778" layer="95"/>
+<pinref part="C1" gate="G$1" pin="1"/>
+<wire x1="393.7" y1="86.36" x2="393.7" y2="91.44" width="0.1524" layer="91"/>
+<junction x="393.7" y="91.44"/>
 </segment>
 <segment>
@@
 <wire x1="365.76" y1="157.48" x2="365.76" y2="160.02" width="0.1524" layer="91"/>
 <label x="365.76" y="160.02" size="1.778" layer="95"/>
+<junction x="365.76" y="157.48"/>
 </segment>
 <segment>
@@
 <wire x1="541.02" y1="459.74" x2="541.02" y2="454.66" width="0.1524" layer="91"/>
 <label x="543.56" y="454.66" size="1.778" layer="95"/>
+<junction x="541.02" y="459.74"/>
 </segment>
 <segment>
@@
 <wire x1="106.68" y1="238.76" x2="114.3" y2="238.76" width="0.1524" layer="91"/>
 <label x="111.76" y="238.76" size="1.778" layer="95"/>
-</segment>
-<segment>
-<wire x1="-40.64" y1="266.7" x2="-27.94" y2="266.7" width="0.1524" layer="91"/>
 </segment>
 <segment>
@@
 <wire x1="482.6" y1="287.02" x2="490.22" y2="287.02" width="0.1524" layer="91"/>
 <label x="482.6" y="287.02" size="1.778" layer="95"/>
+<junction x="482.6" y="279.4"/>
 </segment>
 <segment>
@@
 <label x="-96.52" y="271.78" size="1.778" layer="95"/>
 <pinref part="C16" gate="G$1" pin="1"/>
-<junction x="-35.56" y="314.96"/>
 </segment>
 <segment>
@@
 <label x="-76.2" y="175.26" size="1.778" layer="95"/>
 <pinref part="C25" gate="G$1" pin="1"/>
-<junction x="-15.24" y="218.44"/>
 </segment>
 <segment>
@@
 <label x="-60.96" y="78.74" size="1.778" layer="95"/>
 <pinref part="C29" gate="G$1" pin="1"/>
-<junction x="0" y="121.92"/>
 </segment>
 <segment>
@@
 <junction x="53.34" y="30.48"/>
 <pinref part="C42" gate="G$1" pin="1"/>
-<junction x="50.8" y="38.1"/>
+<label x="2.54" y="0" size="1.778" layer="95"/>
 </segment>
 </net>
@@
 <label x="472.44" y="474.98" size="1.778" layer="95"/>
 <wire x1="449.58" y1="464.82" x2="464.82" y2="464.82" width="0.1524" layer="91"/>
+<junction x="464.82" y="464.82"/>
 </segment>
 </net>
@@
 <wire x1="459.74" y1="147.32" x2="459.74" y2="152.4" width="0.1524" layer="91"/>
 <pinref part="R34" gate="G$1" pin="2"/>
-<wire x1="464.82" y1="152.4" x2="467.36" y2="152.4" width="0.1524" layer="91"/>
 <wire x1="467.36" y1="152.4" x2="474.98" y2="152.4" width="0.1524" layer="91"/>
 <wire x1="474.98" y1="152.4" x2="474.98" y2="137.16" width="0.1524" layer="91"/>
@@
 <wire x1="467.36" y1="142.24" x2="467.36" y2="152.4" width="0.1524" layer="91"/>
 <junction x="467.36" y="152.4"/>
-<wire x1="459.74" y1="152.4" x2="464.82" y2="152.4" width="0.1524" layer="91"/>
-<wire x1="464.82" y1="152.4" x2="464.82" y2="154.94" width="0.1524" layer="91"/>
-<label x="464.82" y="154.94" size="1.778" layer="95"/>
+<wire x1="459.74" y1="152.4" x2="467.36" y2="152.4" width="0.1524" layer="91"/>
+<wire x1="467.36" y1="152.4" x2="467.36" y2="154.94" width="0.1524" layer="91"/>
+<label x="467.36" y="154.94" size="1.778" layer="95"/>
 </segment>
 <segment>
@@
 <wire x1="195.58" y1="177.8" x2="208.28" y2="177.8" width="0.1524" layer="91"/>
 <label x="200.66" y="177.8" size="1.778" layer="95"/>
+<junction x="195.58" y="177.8"/>
 </segment>
 <segment>
@@
 <wire x1="195.58" y1="127" x2="208.28" y2="127" width="0.1524" layer="91"/>
 <label x="200.66" y="127" size="1.778" layer="95"/>
+<junction x="195.58" y="127"/>
 </segment>
 <segment>
@@
 <wire x1="137.16" y1="177.8" x2="149.86" y2="177.8" width="0.1524" layer="91"/>
 <label x="144.78" y="177.8" size="1.778" layer="95"/>
+<junction x="137.16" y="177.8"/>
 </segment>
 <segment>
@@
 <wire x1="137.16" y1="152.4" x2="149.86" y2="152.4" width="0.1524" layer="91"/>
 <label x="142.24" y="152.4" size="1.778" layer="95"/>
+<junction x="137.16" y="152.4"/>
 </segment>
 <segment>
@@
 <wire x1="137.16" y1="127" x2="149.86" y2="127" width="0.1524" layer="91"/>
 <label x="142.24" y="127" size="1.778" layer="95"/>
+<junction x="137.16" y="127"/>
 </segment>
 <segment>
@@
 <wire x1="137.16" y1="203.2" x2="149.86" y2="203.2" width="0.1524" layer="91"/>
 <label x="142.24" y="203.2" size="1.778" layer="95"/>
+<junction x="137.16" y="203.2"/>
 </segment>
 <segment>
@@
 <wire x1="195.58" y1="203.2" x2="208.28" y2="203.2" width="0.1524" layer="91"/>
 <label x="200.66" y="203.2" size="1.778" layer="95"/>
+<junction x="195.58" y="203.2"/>
 </segment>
 <segment>
@@
 <wire x1="195.58" y1="152.4" x2="208.28" y2="152.4" width="0.1524" layer="91"/>
 <label x="200.66" y="152.4" size="1.778" layer="95"/>
+<junction x="195.58" y="152.4"/>
 </segment>
 <segment>
@@
 <wire x1="416.56" y1="119.38" x2="406.4" y2="119.38" width="0.1524" layer="91"/>
 <label x="406.4" y="119.38" size="1.778" layer="95"/>
-</segment>
-</net>
-<net name="N$22" class="0">
-<segment>
-<pinref part="C1" gate="G$1" pin="1"/>
-<wire x1="393.7" y1="86.36" x2="393.7" y2="91.44" width="0.1524" layer="91"/>
 </segment>
 </net>
@@
 <pinref part="R61" gate="G$1" pin="2"/>
 <wire x1="-68.58" y1="330.2" x2="-63.5" y2="330.2" width="0.1524" layer="91"/>
+<junction x="-68.58" y="330.2"/>
 </segment>
 </net>
@@
 <pinref part="R72" gate="G$1" pin="2"/>
 <wire x1="-48.26" y1="233.68" x2="-43.18" y2="233.68" width="0.1524" layer="91"/>
+<junction x="-48.26" y="233.68"/>
 </segment>
 </net>
@@
 <pinref part="R83" gate="G$1" pin="2"/>
 <wire x1="-33.02" y1="137.16" x2="-27.94" y2="137.16" width="0.1524" layer="91"/>
+<junction x="-33.02" y="137.16"/>
 </segment>
 </net>
@@
 <pinref part="R94" gate="G$1" pin="2"/>
 <wire x1="17.78" y1="53.34" x2="22.86" y2="53.34" width="0.1524" layer="91"/>
-</segment>
-</net>
+<junction x="17.78" y="53.34"/>
+</segment>
+</net>

Commit message: clean up and bom
Parts:
- removed KICK_Q, KICK_Q1: (no value), gen3:N-MOSFETDPAK
- removed U$10, U$9: MOTOR_BOARD, Kicker:MOTOR_BOARD
- added Q1, Q2: IXFT94N30P3, transistor-power:IXGT6N170
Connections:
- net 12VGND: now also Q1.E, Q2.E; no longer KICK_Q.S, KICK_Q1.S
- net LOWCHIP: now also Q2.C; no longer KICK_Q1.D
- net LOWKICK: now also Q1.C; no longer KICK_Q.D
- net N$3: now also Q2.G; no longer KICK_Q1.G
- net N$8: now also Q1.G; no longer KICK_Q.G
Changed lines of the file:
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@@
 <part name="CLAMP1" library="gen3" deviceset="DIODE-ZENER" device="DO214AC" value="DIODE-ZENERDO214AC"/>
 <part name="CLAMP2" library="gen3" deviceset="DIODE-ZENER" device="DO214AC" value="DIODE-ZENERDO214AC"/>
-<part name="KICK_Q" library="gen3" deviceset="N-MOSFET" device="DPAK"/>
 <part name="CAP/100" library="gen3" deviceset="TEST_PT" device=""/>
 <part name="CAP_SENSE_BUF" library="SparkFun-AnalogIC" deviceset="MCP6291" device="T-E/OT"/>
@@
 <part name="ANDS" library="gen3" deviceset="AND-DUAL" device=""/>
 <part name="KICK" library="gen3" deviceset="JST-2" device="2MM"/>
-<part name="KICK_Q1" library="gen3" deviceset="N-MOSFET" device="DPAK"/>
 <part name="CHIP_FLY" library="gen3" deviceset="DIODE-ZENER" device="DO214AB"/>
 <part name="CHIP" library="gen3" deviceset="JST-2" device="2MM"/>
@@
 <part name="C13" library="SparkFun-Capacitors" deviceset="CAP" device="0805" value="100nF"/>
 <part name="U$13" library="SparkFun-Connectors" deviceset="PHEONIX-SCREW-TERM" device=""/>
-<part name="U$9" library="Kicker" deviceset="MOTOR_BOARD" device=""/>
-<part name="U$10" library="Kicker" deviceset="MOTOR_BOARD" device=""/>
 <part name="U$16" library="IAD-Library" deviceset="VNH5019" device=""/>
 <part name="U$20" library="IAD-Library" deviceset="MOSFET-NCH" device=""/>
@@
 <part name="R95" library="SparkFun-Passives" deviceset="RESISTOR" device="0805-RES" value="1k"/>
 <part name="R96" library="SparkFun-Passives" deviceset="RESISTOR" device="0805-RES" value="1k"/>
+<part name="Q1" library="transistor-power" library_urn="urn:adsk.eagle:library:400" deviceset="IXG?*N170" device="T" package3d_urn="urn:adsk.eagle:package:29509/1" technology="6" value="IXFT94N30P3"/>
+<part name="Q2" library="transistor-power" library_urn="urn:adsk.eagle:library:400" deviceset="IXG?*N170" device="T" package3d_urn="urn:adsk.eagle:package:29509/1" technology="6" value="IXFT94N30P3"/>
 </parts>
 <sheets>
@@
 <attribute name="NAME" x="798.0426" y="335.28" size="1.778" layer="95" rot="MR90"/>
 </instance>
-<instance part="KICK_Q" gate="G$1" x="480.06" y="312.42" smashed="yes">
-<attribute name="NAME" x="486.41" y="314.96" size="0.7" layer="95" font="vector" ratio="10"/>
-<attribute name="VALUE" x="486.41" y="310.896" size="0.7" layer="95" font="vector" ratio="10"/>
-</instance>
 <instance part="CAP/100" gate="G$1" x="853.44" y="342.9" smashed="yes" rot="MR0">
 <attribute name="NAME" x="857.25" y="345.44" size="1.778" layer="95" rot="MR0"/>
@@
 <instance part="KICK" gate="G$1" x="490.22" y="335.28" smashed="yes">
 <attribute name="NAME" x="487.68" y="327.66" size="1.778" layer="95"/>
-</instance>
-<instance part="KICK_Q1" gate="G$1" x="480.06" y="254" smashed="yes">
-<attribute name="NAME" x="486.41" y="256.54" size="0.7" layer="95" font="vector" ratio="10"/>
-<attribute name="VALUE" x="486.41" y="252.476" size="0.7" layer="95" font="vector" ratio="10"/>
 </instance>
 <instance part="CHIP_FLY" gate="G$1" x="480.06" y="274.32" smashed="yes" rot="R90">
@@
 <attribute name="NAME" x="96.52" y="242.062" size="1.778" layer="95"/>
 </instance>
-<instance part="U$9" gate="G$1" x="223.52" y="261.62" smashed="yes" rot="R90"/>
-<instance part="U$10" gate="G$1" x="223.52" y="330.2" smashed="yes" rot="R90"/>
 <instance part="U$16" gate="G$1" x="-60.96" y="287.02" smashed="yes">
 <attribute name="NAME" x="-73.66" y="302.26" size="1.778" layer="96"/>
@@
 <attribute name="NAME" x="44.45" y="11.6586" size="1.778" layer="95"/>
 <attribute name="VALUE" x="44.45" y="6.858" size="1.778" layer="96"/>
+</instance>
+<instance part="Q1" gate="G$1" x="480.06" y="312.42" smashed="yes">
+<attribute name="NAME" x="485.14" y="314.96" size="1.778" layer="95"/>
+<attribute name="VALUE" x="485.14" y="312.42" size="1.778" layer="96"/>
+</instance>
+<instance part="Q2" gate="G$1" x="480.06" y="254" smashed="yes">
+<attribute name="NAME" x="485.14" y="256.54" size="1.778" layer="95"/>
+<attribute name="VALUE" x="485.14" y="254" size="1.778" layer="96"/>
 </instance>
 </instances>
@@
 </segment>
 <segment>
-<pinref part="KICK_Q1" gate="G$1" pin="S"/>
 <wire x1="482.6" y1="248.92" x2="482.6" y2="243.84" width="0.1524" layer="91"/>
 <label x="482.6" y="243.84" size="1.778" layer="95"/>
-</segment>
-<segment>
-<pinref part="KICK_Q" gate="G$1" pin="S"/>
-<wire x1="482.6" y1="307.34" x2="482.6" y2="302.26" width="0.1524" layer="91"/>
+<pinref part="Q2" gate="G$1" pin="E"/>
+</segment>
+<segment>
 <label x="482.6" y="302.26" size="1.778" layer="95"/>
 <label x="482.6" y="302.26" size="1.778" layer="95"/>
+<pinref part="Q1" gate="G$1" pin="E"/>
+<wire x1="482.6" y1="307.34" x2="482.6" y2="302.26" width="0.1524" layer="91"/>
+<junction x="482.6" y="307.34"/>
 </segment>
 <segment>
@@
 <segment>
 <pinref part="R2" gate="G$1" pin="2"/>
-<pinref part="KICK_Q1" gate="G$1" pin="G"/>
 <wire x1="472.44" y1="274.32" x2="474.98" y2="274.32" width="0.1524" layer="91"/>
-<wire x1="474.98" y1="274.32" x2="474.98" y2="251.46" width="0.1524" layer="91"/>
+<wire x1="474.98" y1="274.32" x2="474.98" y2="254" width="0.1524" layer="91"/>
+<pinref part="Q2" gate="G$1" pin="G"/>
+<wire x1="474.98" y1="254" x2="474.98" y2="251.46" width="0.1524" layer="91"/>
+<junction x="474.98" y="254"/>
 </segment>
 </net>
@@
 <wire x1="482.6" y1="266.7" x2="482.6" y2="259.08" width="0.1524" layer="91"/>
 <junction x="482.6" y="266.7"/>
-<pinref part="KICK_Q1" gate="G$1" pin="D"/>
+<pinref part="Q2" gate="G$1" pin="C"/>
 </segment>
 </net>
 <net name="N$8" class="0">
 <segment>
-<pinref part="KICK_Q" gate="G$1" pin="G"/>
 <pinref part="R1" gate="G$1" pin="2"/>
-<wire x1="474.98" y1="309.88" x2="472.44" y2="309.88" width="0.1524" layer="91"/>
+<wire x1="474.98" y1="312.42" x2="472.44" y2="309.88" width="0.1524" layer="91"/>
+<pinref part="Q1" gate="G$1" pin="G"/>
 </segment>
 </net>
@@
 <wire x1="482.6" y1="325.12" x2="485.14" y2="325.12" width="0.1524" layer="91"/>
 <junction x="482.6" y="325.12"/>
-<pinref part="KICK_Q" gate="G$1" pin="D"/>
 <wire x1="482.6" y1="325.12" x2="482.6" y2="317.5" width="0.1524" layer="91"/>
-</segment>
-</net>
+<pinref part="Q1" gate="G$1" pin="C"/>
+</segment>
+</net>
